Commit message: DRC-1998 pulled in Atlas v4 into sim and tried to fix all of the problems dealing with the switch between shoulder pitch to shoulder yaw. Found some errors with the pose of the head, and inertias in the hokuyo joint. Recreated all the sdf's but removed all the old ones from the atlas robot version, leaving only no hands, gazebo, and robotiq. fixed some UI checks for shoulders to check for hands which is still nasty but better. should fixbamboo, was a flakey test

File: Atlas/resources/models/GFE/atlas_description/urdf/atlas_simple_shapes.urdf (robot description, URDF)
Before this commit: robot drc_skeleton, 28 links, 28 joints
Links:
- link l_foot: mass 0.867 -> 1.634
- link l_lglut: mass 0.803 -> 0.69
- link l_talus: mass 0.867 -> 0.1
- link l_uglut: mass 1.51622 -> 0.5166
- link l_uleg: mass 7.227 -> 7.34
- link ltorso: mass 1.62729 -> 1.92
- link mtorso: mass 3.8068 -> 0.55
- link pelvis: mass 12.54638 -> 14.2529
- link r_foot: mass 0.867 -> 1.634
- link r_lglut: mass 0.803 -> 0.69
- link r_talus: mass 0.867 -> 0.1
- link r_uglut: mass 1.51622 -> 0.5166
- link r_uleg: mass 7.227 -> 7.34
- link utorso: mass 15.2272 -> 18.484

File: Atlas/resources/models/GFE/atlas_description/urdf/atlas_v3.urdf (robot description, URDF)
Before this commit: robot drc_skeleton, 32 links, 32 joints
Links:
- added link rear_situational_awareness_camera_link, mass 0.1; visual box size=0.01 0.01 0.01
- added link rear_situational_awareness_camera_optical_frame
- link l_clav: geometry collision mesh filename=package://atlas_description/meshes_v3/l_clav.stl scale=1 1 1; visual mesh filename=package://atlas_description/meshes_v3/l_clav.dae scale=1 1 1
- link l_farm: geometry collision mesh filename=package://atlas_description/meshes_v3/l_farm.stl scale=1 1 1; visual mesh filename=package://atlas_description/meshes_v3/l_farm.dae scale=1 1 1
- link l_foot: geometry collision mesh filename=package://atlas_description/meshes_v3/l_foot.stl scale=1 1 1; visual mesh filename=package://atlas_description/meshes_v3/l_foot.dae scale=1 1 1
- link l_hand: geometry collision mesh filename=package://atlas_description/meshes_v3/l_hand.stl scale=1 1 1; visual mesh filename=package://atlas_description/meshes_v3/l_hand.dae scale=1 1 1
- link l_larm: geometry collision mesh filename=package://atlas_description/meshes_v3/l_larm.stl scale=1 1 1; visual mesh filename=package://atlas_description/meshes_v3/l_larm.dae scale=1 1 1
- link l_lglut: geometry collision mesh filename=package://atlas_description/meshes_v3/l_lglut.stl scale=1 1 1; visual mesh filename=package://atlas_description/meshes_v3/l_lglut.dae scale=1 1 1
- link l_lleg: geometry collision mesh filename=package://atlas_description/meshes_v3/l_lleg.stl scale=1 1 1; visual mesh filename=package://atlas_description/meshes_v3/l_lleg.dae scale=1 1 1
- link l_scap: geometry collision mesh filename=package://atlas_description/meshes_v3/l_scap.stl scale=1 1 1; visual mesh filename=package://atlas_description/meshes_v3/l_scap.dae scale=1 1 1
- link l_talus: geometry collision mesh filename=package://atlas_description/meshes_v3/l_talus.stl scale=1 1 1; visual mesh filename=package://atlas_description/meshes_v3/l_talus.dae scale=1 1 1
- link l_uarm: geometry collision mesh filename=package://atlas_description/meshes_v3/l_uarm.stl scale=1 1 1; visual mesh filename=package://atlas_description/meshes_v3/l_uarm.dae scale=1 1 1
- link l_uglut: geometry collision mesh filename=package://atlas_description/meshes_v3/l_uglut.stl scale=1 1 1; visual mesh filename=package://atlas_description/meshes_v3/l_uglut.dae scale=1 1 1
- link l_uleg: geometry collision mesh filename=package://atlas_description/meshes_v3/l_uleg.stl scale=1 1 1; visual mesh filename=package://atlas_description/meshes_v3/l_uleg.dae scale=1 1 1
- link ltorso: geometry collision mesh filename=package://atlas_description/meshes_v3/ltorso.stl scale=1 1 1; visual mesh filename=package://atlas_description/meshes_v3/ltorso.dae scale=1 1 1
- link mtorso: geometry collision mesh filename=package://atlas_description/meshes_v3/mtorso.stl scale=1 1 1; visual mesh filename=package://atlas_description/meshes_v3/mtorso.dae scale=1 1 1
- link pelvis: geometry collision mesh filename=package://atlas_description/meshes_v3/pelvis.stl scale=1 1 1; visual mesh filename=package://atlas_description/meshes_v3/pelvis.dae scale=1 1 1
- link r_clav: geometry collision mesh filename=package://atlas_description/meshes_v3/r_clav.stl scale=1 1 1; visual mesh filename=package://atlas_description/meshes_v3/r_clav.dae scale=1 1 1
- link r_farm: geometry collision mesh filename=package://atlas_description/meshes_v3/r_farm.stl scale=1 1 1; visual mesh filename=package://atlas_description/meshes_v3/r_farm.dae scale=1 1 1
- link r_foot: geometry collision mesh filename=package://atlas_description/meshes_v3/r_foot.stl scale=1 1 1; visual mesh filename=package://atlas_description/meshes_v3/r_foot.dae scale=1 1 1
- link r_hand: geometry collision mesh filename=package://atlas_description/meshes_v3/r_hand.stl scale=1 1 1; visual mesh filename=package://atlas_description/meshes_v3/r_hand.dae scale=1 1 1
- link r_larm: geometry collision mesh filename=package://atlas_description/meshes_v3/r_larm.stl scale=1 1 1; visual mesh filename=package://atlas_description/meshes_v3/r_larm.dae scale=1 1 1
- link r_lglut: geometry collision mesh filename=package://atlas_description/meshes_v3/r_lglut.stl scale=1 1 1; visual mesh filename=package://atlas_description/meshes_v3/r_lglut.dae scale=1 1 1
- link r_lleg: geometry collision mesh filename=package://atlas_description/meshes_v3/r_lleg.stl scale=1 1 1; visual mesh filename=package://atlas_description/meshes_v3/r_lleg.dae scale=1 1 1
- link r_scap: geometry collision mesh filename=package://atlas_description/meshes_v3/r_scap.stl scale=1 1 1; visual mesh filename=package://atlas_description/meshes_v3/r_scap.dae scale=1 1 1
- link r_talus: geometry collision mesh filename=package://atlas_description/meshes_v3/r_talus.stl scale=1 1 1; visual mesh filename=package://atlas_description/meshes_v3/r_talus.dae scale=1 1 1
- link r_uarm: geometry collision mesh filename=package://atlas_description/meshes_v3/r_uarm.stl scale=1 1 1; visual mesh filename=package://atlas_description/meshes_v3/r_uarm.dae scale=1 1 1
- link r_uglut: geometry collision mesh filename=package://atlas_description/meshes_v3/r_uglut.stl scale=1 1 1; visual mesh filename=package://atlas_description/meshes_v3/r_uglut.dae scale=1 1 1
- link r_uleg: geometry collision mesh filename=package://atlas_description/meshes_v3/r_uleg.stl scale=1 1 1; visual mesh filename=package://atlas_description/meshes_v3/r_uleg.dae scale=1 1 1
- link utorso: geometry collision mesh filename=package://atlas_description/meshes_v3/utorso.stl scale=1 1 1; collision mesh filename=package://atlas_description/meshes_v3/utorso_pack.stl scale=1 1 1
Joints:
- added joint rear_situational_awareness_camera_joint: type fixed, parent utorso, child rear_situational_awareness_camera_link, origin xyz=-0.0026 0.0264 0.6649 rpy=0 0 3.14159
- added joint rear_situational_awareness_camera_optical_frame_joint: type fixed, parent rear_situational_awareness_camera_link, child rear_situational_awareness_camera_optical_frame, origin xyz=0 0 0 rpy=-1.5708 0.0 -1.5708

File: Atlas/resources/models/GFE/atlas_description/urdf/atlas_v3_with_v1_inertia.urdf (robot description, URDF)
Before this commit: robot drc_skeleton, 32 links, 32 joints
Links:
- link l_clav: geometry collision mesh filename=package://atlas_description/meshes_v3/l_clav.stl scale=1 1 1; visual mesh filename=package://atlas_description/meshes_v3/l_clav.DAE scale=1 1 1
- link l_farm: geometry collision mesh filename=package://atlas_description/meshes_v3/l_farm.stl scale=1 1 1; visual mesh filename=package://atlas_description/meshes_v3/l_farm.DAE scale=1 1 1
- link l_foot: geometry collision mesh filename=package://atlas_description/meshes_v3/l_foot.stl scale=1 1 1; visual mesh filename=package://atlas_description/meshes_v3/l_foot.DAE scale=1 1 1
- link l_hand: geometry collision mesh filename=package://atlas_description/meshes_v3/l_hand.stl scale=1 1 1; visual mesh filename=package://atlas_description/meshes_v3/l_hand.DAE scale=1 1 1
- link l_larm: geometry collision mesh filename=package://atlas_description/meshes_v3/l_elbow_rx.stl scale=1 1 1; visual mesh filename=package://atlas_description/meshes_v3/l_elbow_rx.DAE scale=1 1 1
- link l_lglut: geometry collision mesh filename=package://atlas_description/meshes_v3/l_lglut.stl scale=1 1 1; visual mesh filename=package://atlas_description/meshes_v3/l_lglut.DAE scale=1 1 1
- link l_lleg: geometry collision mesh filename=package://atlas_description/meshes_v3/l_lleg.stl scale=1 1 1; visual mesh filename=package://atlas_description/meshes_v3/l_lleg.DAE scale=1 1 1
- link l_scap: geometry collision mesh filename=package://atlas_description/meshes_v3/l_sh_rx.stl scale=1 1 1; visual mesh filename=package://atlas_description/meshes_v3/l_sh_rx.DAE scale=1 1 1
- link l_talus: geometry collision mesh filename=package://atlas_description/meshes_v3/l_talus.stl scale=1 1 1; visual mesh filename=package://atlas_description/meshes_v3/l_talus.DAE scale=1 1 1
- link l_uarm: geometry collision mesh filename=package://atlas_description/meshes_v3/l_elbow_ry.stl scale=1 1 1; visual mesh filename=package://atlas_description/meshes_v3/l_elbow_ry.DAE scale=1 1 1
- link l_uglut: geometry collision mesh filename=package://atlas_description/meshes_v3/l_uglut.stl scale=1 1 1; visual mesh filename=package://atlas_description/meshes_v3/l_uglut.DAE scale=1 1 1
- link l_uleg: geometry collision mesh filename=package://atlas_description/meshes_v3/l_uleg.stl scale=1 1 1; visual mesh filename=package://atlas_description/meshes_v3/l_uleg.DAE scale=1 1 1
- link ltorso: geometry collision mesh filename=package://atlas_description/meshes_v3/ltorso.stl scale=1 1 1; visual mesh filename=package://atlas_description/meshes_v3/ltorso.DAE scale=1 1 1
- link mtorso: geometry collision mesh filename=package://atlas_description/meshes_v3/mtorso.stl scale=1 1 1; visual mesh filename=package://atlas_description/meshes_v3/mtorso.DAE scale=1 1 1
- link pelvis: geometry collision mesh filename=package://atlas_description/meshes_v3/pelvis.stl scale=1 1 1; visual mesh filename=package://atlas_description/meshes_v3/pelvis.DAE scale=1 1 1
- link r_clav: geometry collision mesh filename=package://atlas_description/meshes_v3/r_clav.stl scale=1 1 1; visual mesh filename=package://atlas_description/meshes_v3/r_clav.DAE scale=1 1 1
- link r_farm: geometry collision mesh filename=package://atlas_description/meshes_v3/r_farm.stl scale=1 1 1; visual mesh filename=package://atlas_description/meshes_v3/r_farm.DAE scale=1 1 1
- link r_foot: geometry collision mesh filename=package://atlas_description/meshes_v3/r_foot.stl scale=1 1 1; visual mesh filename=package://atlas_description/meshes_v3/r_foot.DAE scale=1 1 1
- link r_hand: geometry collision mesh filename=package://atlas_description/meshes_v3/r_hand.stl scale=1 1 1; visual mesh filename=package://atlas_description/meshes_v3/r_hand.DAE scale=1 1 1
- link r_larm: geometry collision mesh filename=package://atlas_description/meshes_v3/r_elbow_rx.stl scale=1 1 1; visual mesh filename=package://atlas_description/meshes_v3/r_elbow_rx.DAE scale=1 1 1
- link r_lglut: geometry collision mesh filename=package://atlas_description/meshes_v3/r_lglut.stl scale=1 1 1; visual mesh filename=package://atlas_description/meshes_v3/r_lglut.DAE scale=1 1 1
- link r_lleg: geometry collision mesh filename=package://atlas_description/meshes_v3/r_lleg.stl scale=1 1 1; visual mesh filename=package://atlas_description/meshes_v3/r_lleg.DAE scale=1 1 1
- link r_scap: geometry collision mesh filename=package://atlas_description/meshes_v3/r_sh_rx.stl scale=1 1 1; visual mesh filename=package://atlas_description/meshes_v3/r_sh_rx.DAE scale=1 1 1
- link r_talus: geometry collision mesh filename=package://atlas_description/meshes_v3/r_talus.stl scale=1 1 1; visual mesh filename=package://atlas_description/meshes_v3/r_talus.DAE scale=1 1 1
- link r_uarm: geometry collision mesh filename=package://atlas_description/meshes_v3/r_elbow_ry.stl scale=1 1 1; visual mesh filename=package://atlas_description/meshes_v3/r_elbow_ry.DAE scale=1 1 1
- link r_uglut: geometry collision mesh filename=package://atlas_description/meshes_v3/r_uglut.stl scale=1 1 1; visual mesh filename=package://atlas_description/meshes_v3/r_uglut.DAE scale=1 1 1
- link r_uleg: geometry collision mesh filename=package://atlas_description/meshes_v3/r_uleg.stl scale=1 1 1; visual mesh filename=package://atlas_description/meshes_v3/r_uleg.DAE scale=1 1 1
- link utorso: geometry collision mesh filename=package://atlas_description/meshes_v3/utorso.stl scale=1 1 1; collision mesh filename=package://atlas_description/meshes_v3/utorso_pack.stl scale=1 1 1

File: Atlas/resources/models/GFE/multisense_sl_description/robots/multisense_sl_description.urdf.xacro (robot description, xacro)
@@ -1,3 +1,3 @@
-<robot xmlns:xacro="http://www.ros.org/wiki/xacro" name="atlas" >
+<robot xmlns:xacro="http://www.ros.org/wiki/xacro" name="multisense_sl" >
   <xacro:include filename="$(find multisense_sl_description)/urdf/multisense_sl.urdf" />
 </robot>
