Commit message: NONE: changed the position of "Hand" in WholeBodyIk to be consistent with SDFFullRobotModel. wont fixBamboo

File: DarpaRoboticsChallenge/resources/models/atlas_v4_robotiq.wb.urdf (robot description, URDF)
Before this commit: robot drc_skeleton, 31 links, 30 joints
Joints:
- joint l_ee_fixed_joint: origin xyz=0  0.26  0 rpy=-1.5708 0 1.5708 -> xyz=0  0.10  0 rpy=0 0 1.5708
- joint r_ee_fixed_joint: origin xyz=0 -0.26  0 rpy=1.5708 0 -1.5708 -> xyz=0 -0.10  0 rpy=0 0 -1.5708

Commit message: NONE: refactoring of WholeBodyIkSolver. wont fixBamboo - Fixed the ModifiebleCylinderGrabber thread safety problem - changed API to set and get position of either the Attachment of the gripper or its center.

File: DarpaRoboticsChallenge/resources/models/atlas_v4_robotiq.wb.urdf (robot description, URDF)
Before this commit: robot drc_skeleton, 31 links, 30 joints
Links:
- removed link l_ee_link
- removed link r_ee_link
- added link l_gripper_attachment
- added link l_gripper_palm
- added link r_gripper_attachment
- added link r_gripper_palm
Joints:
- removed joint l_ee_fixed_joint
- added joint l_ee_fixed_joint1: type fixed, parent l_hand, child l_gripper_attachment, origin xyz=0  0.10  0 rpy=0 0 1.5708
- added joint l_ee_fixed_joint2: type fixed, parent l_gripper_attachment, child l_gripper_palm, origin xyz=0.16 0  0 rpy=0 0 0
- added joint r_ee_fixed_joint2: type fixed, parent r_gripper_attachment, child r_gripper_palm, origin xyz=0.16  0  0 rpy=0 0 0
- joint r_ee_fixed_joint: child r_ee_link -> r_gripper_attachment
