Commit message: NONE: URDF modified with up to date mass. will not fixBamboo

File: DarpaRoboticsChallenge/resources/models/atlas_unplugged.wb.urdf (robot description, URDF)
Before this commit: robot drc_skeleton, 33 links, 32 joints
Links:
- link l_clav: mass 3.45 -> 4.466
- link l_foot: mass 2.05 -> 2.41
- link l_larm: mass 2.509 -> 3.248
- link l_lglut: mass 0.866 -> 0.898
- link l_lleg: mass 5.479 -> 4.515
- link l_scap: mass 3.012 -> 3.899
- link l_uarm: mass 3.388 -> 4.386
- link l_ufarm: mass 3.388 -> 4.386
- link l_uglut: mass 0.648 -> 1.959
- link l_uleg: mass 9.209 -> 8.204
- link ltorso: mass 2.409 -> 2.270
- link mtorso: mass 0.69 -> 0.799
- link pelvis: mass 17.882 -> 9.509
- link r_clav: mass 3.45 -> 4.466
- link r_foot: mass 2.05 -> 2.41
- link r_larm: mass 2.509 -> 3.248
- link r_lglut: mass 0.866 -> 0.898
- link r_lleg: mass 5.479 -> 4.515
- link r_scap: mass 3.012 -> 3.899
- link r_uarm: mass 3.388 -> 4.386
- link r_ufarm: mass 3.388 -> 4.386
- link r_uglut: mass 0.648 -> 1.959
- link r_uleg: mass 9.209 -> 8.204
- link utorso: mass 63.73 -> 84.409
