Commit message: DRC-2232: Tweaks and cleanup to make Davide's car worlds with our plugin self-contained in our catkin workspace. Won't fixbamboo. Ticket is done.

File: Atlas/ihmc_gazebo_catkin_ws/src/ihmc_gazebo/urdf/atlas_v4_no_wry2_simpler_shapes.urdf (robot description, URDF)
Before this commit: robot drc_skeleton, 34 links, 34 joints
Links:
- link l_lleg: geometry collision mesh filename=package://ihmc_gazebo/meshes_unplugged/lleg_low.dae scale=1 1 1; visual mesh filename=package://atlas_description/meshes_unplugged/l_lleg.dae scale=1 1 1
- link l_uleg: geometry collision mesh filename=package://ihmc_gazebo/meshes_unplugged/uleg_low.dae scale=1 1 1; visual mesh filename=package://atlas_description/meshes_unplugged/l_uleg.dae scale=1 1 1
- link pelvis: geometry collision mesh filename=package://ihmc_gazebo/meshes_unplugged/pelvis_low.dae scale=1 1 1; visual mesh filename=package://atlas_description/meshes_unplugged/pelvis.dae scale=1 1 1
- link r_lleg: geometry collision mesh filename=package://ihmc_gazebo/meshes_unplugged/lleg_low.dae scale=1 1 1; visual mesh filename=package://atlas_description/meshes_unplugged/r_lleg.dae scale=1 1 1
- link r_uleg: geometry collision mesh filename=package://ihmc_gazebo/meshes_unplugged/uleg_low.dae scale=1 1 1; visual mesh filename=package://atlas_description/meshes_unplugged/r_uleg.dae scale=1 1 1

File: Atlas/ihmc_gazebo_catkin_ws/src/ihmc_gazebo/urdf/ihmc_atlas_v4.urdf.xacro (robot description, xacro)
@@ -1,4 +1,4 @@
 <robot xmlns:xacro="http://www.ros.org/wiki/xacro" name="atlas" >
-    <xacro:include filename="$(find atlas_description)/urdf/atlas_v4_no_wry2_simpler_shapes.urdf" />
+    <xacro:include filename="$(find ihmc_gazebo)/urdf/atlas_v4_no_wry2_simpler_shapes.urdf" />
     <xacro:include filename="$(find ihmc_gazebo)/urdf/ihmc_atlas_v4.gazebo" />
     <xacro:include filename="$(find atlas_description)/urdf/atlas_v4_no_wry2.transmission" />
