Commit message: DRC-2424: updating urdf and adding in 2cm COM offset to match the sdf. won't fixBamboo

File: Atlas/ihmc_gazebo_catkin_ws/src/ihmc_gazebo/urdf/atlas_v4_no_wry2_simple_shapes.urdf (robot description, URDF)
Before this commit: robot drc_skeleton, 34 links, 34 joints
Links:
- removed link rear_situational_awareness_camera_link
- removed link rear_situational_awareness_camera_optical_frame
- link l_clav: mass 3.45 -> 4.466
- link l_foot: mass 2.05 -> 2.41
- link l_larm: mass 2.509 -> 3.248
- link l_lglut: mass 0.866 -> 0.898
- link l_lleg: mass 5.479 -> 4.515; geometry collision cylinder length=0.40 radius=0.07; visual mesh filename=package://atlas_description/meshes_unplugged/l_lleg.dae scale=1 1 1
- link l_scap: mass 3.012 -> 3.899
- link l_uarm: mass 3.388 -> 4.386
- link l_ufarm: mass 3.388 -> 4.386
- link l_uglut: mass 0.648 -> 1.959
- link l_uleg: mass 9.209 -> 8.204; geometry collision box size=0.07 0.038 0.14; collision box size=0.07 0.038 0.15
- link ltorso: mass 2.409 -> 2.270
- link mtorso: mass 0.69 -> 0.799
- link pelvis: mass 17.882 -> 9.509; geometry collision box size=0.1 0.15 0.2; collision cylinder length=0.05 radius=0.16
- link r_clav: mass 3.45 -> 4.466
- link r_foot: mass 2.05 -> 2.41
- link r_larm: mass 2.509 -> 3.248
- link r_lglut: mass 0.866 -> 0.898
- link r_lleg: mass 5.479 -> 4.515; geometry collision cylinder length=0.40 radius=0.07; visual mesh filename=package://atlas_description/meshes_unplugged/r_lleg.dae scale=1 1 1
- link r_scap: mass 3.012 -> 3.899
- link r_uarm: mass 3.388 -> 4.386
- link r_ufarm: mass 3.388 -> 4.386
- link r_uglut: mass 0.648 -> 1.959
- link r_uleg: mass 9.209 -> 8.204; geometry collision box size=0.07 0.038 0.14; collision box size=0.07 0.038 0.15
- link utorso: mass 63.73 -> 84.409
Joints:
- removed joint rear_situational_awareness_camera_joint
- removed joint rear_situational_awareness_camera_optical_frame_joint
- joint l_situational_awareness_camera_joint: origin xyz=0.216409 0.121799 0.406759 rpy=-1.57079633 0 1.30899694 -> xyz=0.155 0.121 0.785 rpy=0 0 1.309
- joint r_situational_awareness_camera_joint: origin xyz=0.216409 -0.121799 0.406759 rpy=1.57079633 0 -1.30899694 -> xyz=0.155 -0.121 0.785 rpy=0 0 -1.309

File: Atlas/ihmc_gazebo_catkin_ws/src/ihmc_gazebo/urdf/ihmc_atlas_v4.urdf.xacro (robot description, xacro)
@@ -1,4 +1,4 @@
 <robot xmlns:xacro="http://www.ros.org/wiki/xacro" name="atlas" >
-    <xacro:include filename="$(find ihmc_gazebo)/urdf/atlas_v4_no_wry2_simpler_shapes.urdf" />
+    <xacro:include filename="$(find ihmc_gazebo)/urdf/atlas_v4_no_wry2_simple_shapes.urdf" />
     <xacro:include filename="$(find ihmc_gazebo)/urdf/ihmc_atlas_v4.gazebo" />
     <xacro:include filename="$(find atlas_description)/urdf/atlas_v4_no_wry2.transmission" />
