Commit message: ROSI-209: Loaded Val A and B models in to SCS, think I found all the strings where names have changed. Adjust hokuyo link inertia in code now instead of the .sdf. Haven't backported any other changes from the .sdf since they've changed so much that diffing is really hard, and they may no longer be necessary. Won't fixbamboo. Pair: Nicolas. #needs-review

File: resources/models/val_description/urdf/valkyrie_A_hw.urdf (robot description, URDF)
Before this commit: robot valkyrie, 70 links, 69 joints
Links:
- removed link LeftAnklePitchLink
- removed link LeftCOP_Frame
- removed link LeftElbowPitchLink
- removed link LeftFoot
- removed link LeftFootSixAxis_Frame
- removed link LeftForearmLink
- removed link LeftHazardCamera_Frame
- removed link LeftHipPitchLink
- removed link LeftHipRollLink
- removed link LeftHipYawLink
- removed link LeftIndexFingerPitch1Link
- removed link LeftIndexFingerPitch2Link
- removed link LeftIndexFingerPitch3Link
- removed link LeftKneePitchLink
- removed link LeftMiddleFingerPitch1Link
- removed link LeftMiddleFingerPitch2Link
- removed link LeftMiddleFingerPitch3Link
- removed link LeftPalm
- removed link LeftPelvisIMU_Frame
- removed link LeftPinkyPitch1Link
- removed link LeftPinkyPitch2Link
- removed link LeftPinkyPitch3Link
- removed link LeftShoulderPitchLink
- removed link LeftShoulderRollLink
- removed link LeftShoulderYawLink
- removed link LeftThumbPitch1Link
- removed link LeftThumbPitch2Link
- removed link LeftThumbPitch3Link
- removed link LeftThumbRollLink
- removed link LeftTorsoIMU_Frame
- removed link LeftWristRollLink
- removed link LowerNeckPitchLink
- removed link NeckYawLink
- removed link Pelvis
- removed link RightAnklePitchLink
- removed link RightCOP_Frame
- removed link RightElbowPitchLink
- removed link RightFoot
- removed link RightFootSixAxis_Frame
- removed link RightForearmLink
- removed link RightHazardCamera_Frame
- removed link RightHipPitchLink
- removed link RightHipRollLink
- removed link RightHipYawLink
- removed link RightIndexFingerPitch1Link
- removed link RightIndexFingerPitch2Link
- removed link RightIndexFingerPitch3Link
- removed link RightKneePitchLink
- removed link RightMiddleFingerPitch1Link
- removed link RightMiddleFingerPitch2Link
- removed link RightMiddleFingerPitch3Link
- removed link RightPalm
- removed link RightPelvisIMU_Frame
- removed link RightPinkyPitch1Link
- removed link RightPinkyPitch2Link
- removed link RightPinkyPitch3Link
- removed link RightShoulderPitchLink
- removed link RightShoulderRollLink
- removed link RightShoulderYawLink
- removed link RightThumbPitch1Link
- removed link RightThumbPitch2Link
- removed link RightThumbPitch3Link
- removed link RightThumbRollLink
- removed link RightTorsoIMU_Frame
- removed link RightWristRollLink
- removed link Torso
- removed link TorsoPitchLink
- removed link TorsoYawLink
- removed link UpperNeckPitchLink
- added link leftAnklePitchLink, mass 0.06; collision mesh filename=package://val_description/model/meshes/legs/lj5.dae; visual mesh filename=package://val_description/model/meshes/legs/lj5.dae
- added link leftCOP_Frame, mass 0.1
- added link leftElbowPitchLink, mass 1.83; collision mesh filename=package://val_description/model/meshes/arms/aj4_left.dae; visual mesh filename=package://val_description/model/meshes/arms/aj4_left.dae
- added link leftFoot, mass 3.255; collision box size=0.27 0.16 0.064; visual mesh filename=package://val_description/model/meshes/legs/foot.dae
- added link leftFootSixAxis_Frame, mass 1e-07
- added link leftForearmLink, mass 2.476; collision mesh filename=package://val_description/model/meshes/arms/aj5_left.dae; visual mesh filename=package://val_description/model/meshes/arms/aj5_left.dae
- added link leftHazardCamera_Frame, mass 1e-07
- added link leftHipPitchLink, mass 10.2; collision mesh filename=package://val_description/model/meshes/legs/lj3_left.dae; visual mesh filename=package://val_description/model/meshes/legs/lj3_left.dae
- added link leftHipRollLink, mass 3.665; collision mesh filename=package://val_description/model/meshes/legs/lj2_left.dae; visual mesh filename=package://val_description/model/meshes/legs/lj2_left.dae
- added link leftHipYawLink, mass 2.39; collision mesh filename=package://val_description/model/meshes/legs/lj1_left.dae; visual mesh filename=package://val_description/model/meshes/legs/lj1_left.dae
- added link leftIndexFingerPitch1Link, mass 0.02; collision mesh filename=package://val_description/model/meshes/fingers/indexj1_left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; visual mesh filename=package://val_description/model/meshes/fingers/indexj1_left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
- added link leftIndexFingerPitch2Link, mass 0.018; collision mesh filename=package://val_description/model/meshes/fingers/indexj2_left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; visual mesh filename=package://val_description/model/meshes/fingers/indexj2_left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
- added link leftIndexFingerPitch3Link, mass 0.01; collision mesh filename=package://val_description/model/meshes/fingers/indexj3_left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; visual mesh filename=package://val_description/model/meshes/fingers/indexj3_left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
- added link leftKneePitchLink, mass 6.6; collision mesh filename=package://val_description/model/meshes/legs/lj4_left.dae; visual mesh filename=package://val_description/model/meshes/legs/lj4_left.dae
- added link leftMiddleFingerPitch1Link, mass 0.02; collision mesh filename=package://val_description/model/meshes/fingers/middlej1_lef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; visual mesh filename=package://val_description/model/meshes/fingers/middlej1_lef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
- added link leftMiddleFingerPitch2Link, mass 0.011; collision mesh filename=package://val_description/model/meshes/fingers/middlej2_lef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; visual mesh filename=package://val_description/model/meshes/fingers/middlej2_lef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
- added link leftMiddleFingerPitch3Link, mass 0.006; collision mesh filename=package://val_description/model/meshes/fingers/middlej3_lef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; visual mesh filename=package://val_description/model/meshes/fingers/middlej3_lef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
- added link leftPalm, mass 0.712; collision mesh filename=package://val_description/model/meshes/arms/palm_left.dae; visual mesh filename=package://val_description/model/meshes/arms/palm_left.dae
- added link leftPelvisIMU_Frame, mass 1e-07
- added link leftPinkyPitch1Link, mass 0.02; collision mesh filename=package://val_description/model/meshes/fingers/pinkyj1_left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; visual mesh filename=package://val_description/model/meshes/fingers/pinkyj1_left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
- added link leftPinkyPitch2Link, mass 0.011; collision mesh filename=package://val_description/model/meshes/fingers/pinkyj2_left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; visual mesh filename=package://val_description/model/meshes/fingers/pinkyj2_left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
- added link leftPinkyPitch3Link, mass 0.006; collision mesh filename=package://val_description/model/meshes/fingers/pinkyj3_left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; visual mesh filename=package://val_description/model/meshes/fingers/pinkyj3_left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
- added link leftShoulderPitchLink, mass 2.65; collision mesh filename=package://val_description/model/meshes/arms/aj1_left.dae; visual mesh filename=package://val_description/model/meshes/arms/aj1_left.dae
- added link leftShoulderRollLink, mass 3.97; collision mesh filename=package://val_description/model/meshes/arms/aj2_left.dae; visual mesh filename=package://val_description/model/meshes/arms/aj2_left.dae
- added link leftShoulderYawLink, mass 3.085; collision mesh filename=package://val_description/model/meshes/arms/aj3_left.dae; visual mesh filename=package://val_description/model/meshes/arms/aj3_left.dae
- added link leftThumbPitch1Link, mass 0.02; collision mesh filename=package://val_description/model/meshes/fingers/thumbj2_left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; visual mesh filename=package://val_description/model/meshes/fingers/thumbj2_left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
- added link leftThumbPitch2Link, mass 0.013; collision mesh filename=package://val_description/model/meshes/fingers/thumbj3_left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; visual mesh filename=package://val_description/model/meshes/fingers/thumbj3_left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
- added link leftThumbPitch3Link, mass 0.006; collision mesh filename=package://val_description/model/meshes/fingers/thumbj4_left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; visual mesh filename=package://val_description/model/meshes/fingers/thumbj4_left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
- added link leftThumbRollLink, mass 0.017; collision mesh filename=package://val_description/model/meshes/fingers/thumbj1_left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; visual mesh filename=package://val_description/model/meshes/fingers/thumbj1_left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
- added link leftTorsoIMU_Frame, mass 1e-07
- added link leftWristRollLink, mass 0.14; collision mesh filename=package://val_description/model/meshes/arms/aj6_left.dae; visual mesh filename=package://val_description/model/meshes/arms/aj6_left.dae
- added link lowerNeckPitchLink, mass 1.05; collision mesh filename=package://val_description/model/meshes/head/neckj1.dae; visual mesh filename=package://val_description/model/meshes/head/neckj1.dae
- added link neckYawLink, mass 1.4; collision mesh filename=package://val_description/model/meshes/head/neckj2.dae; visual mesh filename=package://val_description/model/meshes/head/neckj2.dae
- added link pelvis, mass 8.22; collision mesh filename=package://val_description/model/meshes/pelvis/pelvis.dae; visual mesh filename=package://val_description/model/meshes/pelvis/pelvis.dae
- added link rightAnklePitchLink, mass 0.06; collision mesh filename=package://val_description/model/meshes/legs/lj5.dae; visual mesh filename=package://val_description/model/meshes/legs/lj5.dae
- added link rightCOP_Frame, mass 0.1
- added link rightElbowPitchLink, mass 1.83; collision mesh filename=package://val_description/model/meshes/arms/aj4_right.dae; visual mesh filename=package://val_description/model/meshes/arms/aj4_right.dae
- added link rightFoot, mass 3.255; collision box size=0.27 0.16 0.064; visual mesh filename=package://val_description/model/meshes/legs/foot.dae
- added link rightFootSixAxis_Frame, mass 1e-07
- added link rightForearmLink, mass 2.476; collision mesh filename=package://val_description/model/meshes/arms/aj5_right.dae; visual mesh filename=package://val_description/model/meshes/arms/aj5_right.dae
- added link rightHazardCamera_Frame, mass 1e-07
- added link rightHipPitchLink, mass 10.2; collision mesh filename=package://val_description/model/meshes/legs/lj3_right.dae; visual mesh filename=package://val_description/model/meshes/legs/lj3_right.dae
- added link rightHipRollLink, mass 3.665; collision mesh filename=package://val_description/model/meshes/legs/lj2_right.dae; visual mesh filename=package://val_description/model/meshes/legs/lj2_right.dae
- added link rightHipYawLink, mass 2.39; collision mesh filename=package://val_description/model/meshes/legs/lj1_right.dae; visual mesh filename=package://val_description/model/meshes/legs/lj1_right.dae
- added link rightIndexFingerPitch1Link, mass 0.02; collision mesh filename=package://val_description/model/meshes/fingers/indexj1_righ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; visual mesh filename=package://val_description/model/meshes/fingers/indexj1_righ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
- added link rightIndexFingerPitch2Link, mass 0.018; collision mesh filename=package://val_description/model/meshes/fingers/indexj2_righ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; visual mesh filename=package://val_description/model/meshes/fingers/indexj2_righ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
- added link rightIndexFingerPitch3Link, mass 0.01; collision mesh filename=package://val_description/model/meshes/fingers/indexj3_righ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; visual mesh filename=package://val_description/model/meshes/fingers/indexj3_righ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
- added link rightKneePitchLink, mass 6.6; collision mesh filename=package://val_description/model/meshes/legs/lj4_right.dae; visual mesh filename=package://val_description/model/meshes/legs/lj4_right.dae
- added link rightMiddleFingerPitch1Link, mass 0.02; collision mesh filename=package://val_description/model/meshes/fingers/middlej1_rig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; visual mesh filename=package://val_description/model/meshes/fingers/middlej1_rig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
- added link rightMiddleFingerPitch2Link, mass 0.011; collision mesh filename=package://val_description/model/meshes/fingers/middlej2_rig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; visual mesh filename=package://val_description/model/meshes/fingers/middlej2_rig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
- added link rightMiddleFingerPitch3Link, mass 0.006; collision mesh filename=package://val_description/model/meshes/fingers/middlej3_rig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; visual mesh filename=package://val_description/model/meshes/fingers/middlej3_rig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
- added link rightPalm, mass 0.712; collision mesh filename=package://val_description/model/meshes/arms/palm_right.dae; visual mesh filename=package://val_description/model/meshes/arms/palm_right.dae
- added link rightPelvisIMU_Frame, mass 1e-07
- added link rightPinkyPitch1Link, mass 0.02; collision mesh filename=package://val_description/model/meshes/fingers/pinkyj1_righ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; visual mesh filename=package://val_description/model/meshes/fingers/pinkyj1_righ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
- added link rightPinkyPitch2Link, mass 0.011; collision mesh filename=package://val_description/model/meshes/fingers/pinkyj2_righ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; visual mesh filename=package://val_description/model/meshes/fingers/pinkyj2_righ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
- added link rightPinkyPitch3Link, mass 0.006; collision mesh filename=package://val_description/model/meshes/fingers/pinkyj3_righ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; visual mesh filename=package://val_description/model/meshes/fingers/pinkyj3_righ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
- added link rightShoulderPitchLink, mass 2.65; collision mesh filename=package://val_description/model/meshes/arms/aj1_right.dae; visual mesh filename=package://val_description/model/meshes/arms/aj1_right.dae
- added link rightShoulderRollLink, mass 3.97; collision mesh filename=package://val_description/model/meshes/arms/aj2_right.dae; visual mesh filename=package://val_description/model/meshes/arms/aj2_right.dae
- added link rightShoulderYawLink, mass 3.085; collision mesh filename=package://val_description/model/meshes/arms/aj3_right.dae; visual mesh filename=package://val_description/model/meshes/arms/aj3_right.dae
- added link rightThumbPitch1Link, mass 0.02; collision mesh filename=package://val_description/model/meshes/fingers/thumbj2_righ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; visual mesh filename=package://val_description/model/meshes/fingers/thumbj2_righ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
- added link rightThumbPitch2Link, mass 0.013; collision mesh filename=package://val_description/model/meshes/fingers/thumbj3_righ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; visual mesh filename=package://val_description/model/meshes/fingers/thumbj3_righ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
- added link rightThumbPitch3Link, mass 0.006; collision mesh filename=package://val_description/model/meshes/fingers/thumbj4_righ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; visual mesh filename=package://val_description/model/meshes/fingers/thumbj4_righ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
- added link rightThumbRollLink, mass 0.017; collision mesh filename=package://val_description/model/meshes/fingers/thumbj1_righ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; visual mesh filename=package://val_description/model/meshes/fingers/thumbj1_righ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
- added link rightTorsoIMU_Frame, mass 1e-07
- added link rightWristRollLink, mass 0.14; collision mesh filename=package://val_description/model/meshes/arms/aj6_right.dae; visual mesh filename=package://val_description/model/meshes/arms/aj6_right.dae
- added link torso, mass 39.47; collision mesh filename=package://val_description/model/meshes/torso/torso.dae; visual mesh filename=package://val_description/model/meshes/torso/torso.dae
- added link torsoPitchLink, mass 0.1; collision mesh filename=package://val_description/model/meshes/torso/torsopitch.dae; visual mesh filename=package://val_description/model/meshes/torso/torsopitch.dae
- added link torsoYawLink, mass 0.5; collision mesh filename=package://val_description/model/meshes/torso/torsoyaw.dae; visual mesh filename=package://val_description/model/meshes/torso/torsoyaw.dae
- added link upperNeckPitchLink, mass 4.59; collision mesh filename=package://val_description/model/meshes/head/head_multisense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; visual mesh filename=package://val_description/model/meshes/head/head_multisense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
Joints:
- removed joint LeftAnklePitch
- removed joint LeftAnkleRoll
- removed joint LeftCOP_Offset
- removed joint LeftElbowPitch
- removed joint LeftFootSixAxis_Offset
- removed joint LeftForearmYaw
- removed joint LeftHazardCamera_Offset
- removed joint LeftHipPitch
- removed joint LeftHipRoll
- removed joint LeftHipYaw
- removed joint LeftIndexFingerPitch1
- removed joint LeftIndexFingerPitch2
- removed joint LeftIndexFingerPitch3
- removed joint LeftKneePitch
- removed joint LeftMiddleFingerPitch1
- removed joint LeftMiddleFingerPitch2
- removed joint LeftMiddleFingerPitch3
- removed joint LeftPelvisIMU_Offset
- removed joint LeftPinkyPitch1
- removed joint LeftPinkyPitch2
- removed joint LeftPinkyPitch3
- removed joint LeftShoulderPitch
- removed joint LeftShoulderRoll
- removed joint LeftShoulderYaw
- removed joint LeftThumbPitch1
- removed joint LeftThumbPitch2
- removed joint LeftThumbPitch3
- removed joint LeftThumbRoll
- removed joint LeftTorsoIMU_Offset
- removed joint LeftWristPitch
- removed joint LeftWristRoll
- removed joint LowerNeckPitch
- removed joint NeckYaw
- removed joint RightAnklePitch
- removed joint RightAnkleRoll
- removed joint RightCOP_Offset
- removed joint RightElbowPitch
- removed joint RightFootSixAxis_Offset
- removed joint RightForearmYaw
- removed joint RightHazardCamera_Offset
- removed joint RightHipPitch
- removed joint RightHipRoll
- removed joint RightHipYaw
- removed joint RightIndexFingerPitch1
- removed joint RightIndexFingerPitch2
- removed joint RightIndexFingerPitch3
- removed joint RightKneePitch
- removed joint RightMiddleFingerPitch1
- removed joint RightMiddleFingerPitch2
- removed joint RightMiddleFingerPitch3
- removed joint RightPelvisIMU_Offset
- removed joint RightPinkyPitch1
- removed joint RightPinkyPitch2
- removed joint RightPinkyPitch3
- removed joint RightShoulderPitch
- removed joint RightShoulderRoll
- removed joint RightShoulderYaw
- removed joint RightThumbPitch1
- removed joint RightThumbPitch2
- removed joint RightThumbPitch3
- removed joint RightThumbRoll
- removed joint RightTorsoIMU_Offset
- removed joint RightWristPitch
- removed joint RightWristRoll
- removed joint TorsoPitch
- removed joint TorsoRoll
- removed joint TorsoYaw
- removed joint UpperNeckPitch
- added joint leftAnklePitch: type revolute, parent leftKneePitchLink, child leftAnklePitchLink, origin xyz=-0.0102381 0.0 -0.40627 rpy=0.0 0.0 0.0, axis 0 1 0, limit lower=-0.8644 upper=0.875 effort=205 velocity=11
- added joint leftAnkleRoll: type revolute, parent leftAnklePitchLink, child leftFoot, origin xyz=0.0 0.0 0.0 rpy=0.0 0.0 0.0, axis 1 0 0, limit lower=-0.349 upper=0.348 effort=205 velocity=11
- added joint leftCOP_Offset: type fixed, parent leftFoot, child leftCOP_Frame, origin xyz=0.0189 0.0 -0.0783 rpy=0.0 0.13 0.0, axis 0 0 1
- added joint leftElbowPitch: type revolute, parent leftShoulderYawLink, child leftElbowPitchLink, origin xyz=0.0254 0.33 0.0 rpy=0.0 0.0 0.0, axis 0 0 1, limit lower=-2.174 upper=0.12 effort=65 velocity=11.5
- added joint leftFootSixAxis_Offset: type fixed, parent leftFoot, child leftFootSixAxis_Frame, origin xyz=0.0215646 0.0 -0.051054 rpy=3.14 0.0 -1.047, axis 0 0 1
- added joint leftForearmYaw: type revolute, parent leftElbowPitchLink, child leftForearmLink, origin xyz=-0.0254 0 0 rpy=0.0 0.0 0.0, axis 0 1 0, limit lower=-2.019 upper=3.14 effort=26 velocity=5
- added joint leftHazardCamera_Offset: type fixed, parent torso, child leftHazardCamera_Frame, origin xyz=0.0345 0.0406 0.1135 rpy=1.57 0.0 1.57, axis 0 0 1
- added joint leftHipPitch: type revolute, parent leftHipRollLink, child leftHipPitchLink, origin xyz=0.0 0.0 -0.0609 rpy=0.0 0.0 0.0, axis 0 1 0, limit lower=-2.42 upper=1.619 effort=350 velocity=6.11
- added joint leftHipRoll: type revolute, parent leftHipYawLink, child leftHipRollLink, origin xyz=0.0 0.0 0.0 rpy=0.0 0.0 0.0, axis 1 0 0, limit lower=-0.467 upper=0.5515 effort=350 velocity=7
- added joint leftHipYaw: type revolute, parent pelvis, child leftHipYawLink, origin xyz=0.0 0.1016 -0.1853 rpy=0.0 0.0 0.0, axis 0 0 1, limit lower=-0.4141 upper=1.1 effort=190 velocity=5.89
- added joint leftIndexFingerPitch1: type revolute, parent leftPalm, child leftIndexFingerPitch1Link, origin xyz=0.0022 0.0976 0.0235 rpy=0.1745 0.0 0.0, axis 0 0 1, limit lower=-1.57 upper=-0.0 effort=10 velocity=1
- added joint leftIndexFingerPitch2: type revolute, parent leftIndexFingerPitch1Link, child leftIndexFingerPitch2Link, origin xyz=0.0 0.0381 0.0 rpy=0.0 0.0 0.0, axis 0 0 1, limit lower=-1.658 upper=-0.0 effort=10 velocity=1
- added joint leftIndexFingerPitch3: type revolute, parent leftIndexFingerPitch2Link, child leftIndexFingerPitch3Link, origin xyz=0.0 0.0229 0 rpy=0.0 0.0 0.0, axis 0 0 1, limit lower=-1.92 upper=-0.0 effort=10 velocity=1
- added joint leftKneePitch: type revolute, parent leftHipPitchLink, child leftKneePitchLink, origin xyz=0.000112225 0.0361046 -0.430959 rpy=0.0 0.0 0.0, axis 0 1 0, limit lower=-0.083 upper=2.057 effort=350 velocity=6.11
- added joint leftMiddleFingerPitch1: type revolute, parent leftPalm, child leftMiddleFingerPitch1Link, origin xyz=0.0022 0.097 -0.0119 rpy=-0.1222 0.0 0.0, axis 0 0 1, limit lower=-1.658 upper=-0.0 effort=10 velocity=1
- added joint leftMiddleFingerPitch2: type revolute, parent leftMiddleFingerPitch1Link, child leftMiddleFingerPitch2Link, origin xyz=0.0 0.0381 0.0 rpy=0.0 0.0 0.0, axis 0 0 1, limit lower=-1.92 upper=-0.0 effort=10 velocity=1
- added joint leftMiddleFingerPitch3: type revolute, parent leftMiddleFingerPitch2Link, child leftMiddleFingerPitch3Link, origin xyz=0.0 0.0229 0.0 rpy=0.0 0.0 0.0, axis 0 0 1, limit lower=-1.57 upper=-0.0 effort=10 velocity=1
- added joint leftPelvisIMU_Offset: type fixed, parent pelvis, child leftPelvisIMU_Frame, origin xyz=0.0515 0.115 -0.042 rpy=1.57 0 -1.274, axis 0 0 1
- added joint leftPinkyPitch1: type revolute, parent leftPalm, child leftPinkyPitch1Link, origin xyz=0.0022 0.0838 -0.041 rpy=-0.1222 0.0 0.0, axis 0 0 1, limit lower=-1.57 upper=-0.0 effort=10 velocity=1
- added joint leftPinkyPitch2: type revolute, parent leftPinkyPitch1Link, child leftPinkyPitch2Link, origin xyz=0.0 0.0381 0.0 rpy=0.0 0.0 0.0, axis 0 0 1, limit lower=-1.658 upper=-0.0 effort=10 velocity=1
- added joint leftPinkyPitch3: type revolute, parent leftPinkyPitch2Link, child leftPinkyPitch3Link, origin xyz=0.0 0.0229 0.0 rpy=0.0 0.0 0.0, axis 0 0 1, limit lower=-1.92 upper=-0.0 effort=10 velocity=1
- added joint leftShoulderPitch: type revolute, parent torso, child leftShoulderPitchLink, origin xyz=-0.0316 0.0 0.2984 rpy=0.0 0.0 0.0, axis 0 1 0, limit lower=-2.85 upper=2.0 effort=190 velocity=5.89
- added joint leftShoulderRoll: type revolute, parent leftShoulderPitchLink, child leftShoulderRollLink, origin xyz=0.0 0.2499 0.0 rpy=0.0 0.0 0.0, axis 1 0 0, limit lower=-1.519 upper=1.266 effort=190 velocity=5.89
- added joint leftShoulderYaw: type revolute, parent leftShoulderRollLink, child leftShoulderYawLink, origin xyz=0.0 0.0 0.0 rpy=0.0 0.0 0.0, axis 0 1 0, limit lower=-3.1 upper=2.18 effort=65 velocity=11.5
- added joint leftThumbPitch1: type revolute, parent leftThumbRollLink, child leftThumbPitch1Link, origin xyz=0.0 0.0 0.0229 rpy=0.3491 0.0 0.0, axis 1 0 0, limit lower=-1.658 upper=-0.0 effort=10 velocity=1
- added joint leftThumbPitch2: type revolute, parent leftThumbPitch1Link, child leftThumbPitch2Link, origin xyz=0.0 0.0066 0.0375 rpy=0.0 0.0 0.0, axis 1 0 0, limit lower=-1.92 upper=-0.0 effort=10 velocity=1
- added joint leftThumbPitch3: type revolute, parent leftThumbPitch2Link, child leftThumbPitch3Link, origin xyz=0.0 0.0049 0.0275 rpy=0.0 0.0 0.0, axis 1 0 0, limit lower=-1.57 upper=-0.0 effort=10 velocity=1
- added joint leftThumbRoll: type revolute, parent leftPalm, child leftThumbRollLink, origin xyz=0.0049 0.0351 0.0228 rpy=-0.3491 0.0 0.0, axis 0 1 0, limit lower=0.0 upper=2.356 effort=10 velocity=1
- added joint leftTorsoIMU_Offset: type fixed, parent torso, child leftTorsoIMU_Frame, origin xyz=-0.047 0.134 0.363 rpy=1.57 0.0 3.14, axis 0 0 1
- added joint leftWristPitch: type revolute, parent leftWristRollLink, child leftPalm, origin xyz=0.0 0.0 0.0 rpy=0.0 0.0 0.0, axis 0 0 1, limit lower=-0.36 upper=0.49 effort=14 velocity=1
- added joint leftWristRoll: type revolute, parent leftForearmLink, child leftWristRollLink, origin xyz=0.0 0.2871 0.0 rpy=0.0 0.0 0.0, axis 1 0 0, limit lower=-0.62 upper=0.625 effort=14 velocity=1
- added joint lowerNeckPitch: type revolute, parent torso, child lowerNeckPitchLink, origin xyz=0.0203518 0.0 0.33845 rpy=0.0 0.0 0.0, axis 0 1 0, limit lower=0 upper=1.162 effort=26 velocity=5
- added joint neckYaw: type revolute, parent lowerNeckPitchLink, child neckYawLink, origin xyz=-0.051924 0.0 0.0 rpy=0.0 0.0 0.0, axis 0 0 1, limit lower=-1.04719755 upper=1.04719755 effort=26 velocity=5
- added joint rightAnklePitch: type revolute, parent rightKneePitchLink, child rightAnklePitchLink, origin xyz=-0.0102381 0.0 -0.40627 rpy=0.0 0.0 0.0, axis 0 1 0, limit lower=-0.8644 upper=0.875 effort=205 velocity=11
- added joint rightAnkleRoll: type revolute, parent rightAnklePitchLink, child rightFoot, origin xyz=0.0 0.0 0.0 rpy=0.0 0.0 0.0, axis 1 0 0, limit lower=-0.349 upper=0.348 effort=205 velocity=11
- added joint rightCOP_Offset: type fixed, parent rightFoot, child rightCOP_Frame, origin xyz=0.0189 0.0 -0.0783 rpy=0.0 0.13 0.0, axis 0 0 1
- added joint rightElbowPitch: type revolute, parent rightShoulderYawLink, child rightElbowPitchLink, origin xyz=0.0254 -0.33 0.0 rpy=0.0 0.0 0.0, axis 0 0 1, limit lower=-0.12 upper=2.174 effort=65 velocity=11.5
- added joint rightFootSixAxis_Offset: type fixed, parent rightFoot, child rightFootSixAxis_Frame, origin xyz=0.0215646 0.0 -0.051054 rpy=3.14 0.0 -1.047, axis 0 0 1
- added joint rightForearmYaw: type revolute, parent rightElbowPitchLink, child rightForearmLink, origin xyz=-0.0254 0 0 rpy=0.0 0.0 0.0, axis 0 1 0, limit lower=-2.019 upper=3.14 effort=26 velocity=5
- added joint rightHazardCamera_Offset: type fixed, parent torso, child rightHazardCamera_Frame, origin xyz=0.0345 -0.0406 0.1135 rpy=1.57 0.0 1.57, axis 0 0 1
- added joint rightHipPitch: type revolute, parent rightHipRollLink, child rightHipPitchLink, origin xyz=0.0 0.0 -0.0609 rpy=0.0 0.0 0.0, axis 0 1 0, limit lower=-2.42 upper=1.619 effort=350 velocity=6.11
- added joint rightHipRoll: type revolute, parent rightHipYawLink, child rightHipRollLink, origin xyz=0.0 0.0 0.0 rpy=0.0 0.0 0.0, axis 1 0 0, limit lower=-0.5515 upper=0.467 effort=350 velocity=7
- added joint rightHipYaw: type revolute, parent pelvis, child rightHipYawLink, origin xyz=0.0 -0.1016 -0.1853 rpy=0.0 0.0 0.0, axis 0 0 1, limit lower=-1.1 upper=0.4141 effort=190 velocity=5.89
- added joint rightIndexFingerPitch1: type revolute, parent rightPalm, child rightIndexFingerPitch1Link, origin xyz=0.0022 -0.0976 0.0235 rpy=-0.1745 0.0 0.0, axis 0 0 1, limit lower=0.0 upper=1.57 effort=10 velocity=1
- added joint rightIndexFingerPitch2: type revolute, parent rightIndexFingerPitch1Link, child rightIndexFingerPitch2Link, origin xyz=0.0 -0.0381 0.0 rpy=0.0 0.0 0.0, axis 0 0 1, limit lower=0.0 upper=1.658 effort=10 velocity=1
- added joint rightIndexFingerPitch3: type revolute, parent rightIndexFingerPitch2Link, child rightIndexFingerPitch3Link, origin xyz=0.0 -0.0229 0 rpy=0.0 0.0 0.0, axis 0 0 1, limit lower=0.0 upper=1.92 effort=10 velocity=1
- added joint rightKneePitch: type revolute, parent rightHipPitchLink, child rightKneePitchLink, origin xyz=0.000112225 -0.0361046 -0.430959 rpy=0.0 0.0 0.0, axis 0 1 0, limit lower=-0.083 upper=2.057 effort=350 velocity=6.11
- added joint rightMiddleFingerPitch1: type revolute, parent rightPalm, child rightMiddleFingerPitch1Link, origin xyz=0.0022 -0.097 -0.0119 rpy=0.1222 0.0 0.0, axis 0 0 1, limit lower=0.0 upper=1.658 effort=10 velocity=1
- added joint rightMiddleFingerPitch2: type revolute, parent rightMiddleFingerPitch1Link, child rightMiddleFingerPitch2Link, origin xyz=0.0 -0.0381 0.0 rpy=0.0 0.0 0.0, axis 0 0 1, limit lower=0.0 upper=1.92 effort=10 velocity=1
- added joint rightMiddleFingerPitch3: type revolute, parent rightMiddleFingerPitch2Link, child rightMiddleFingerPitch3Link, origin xyz=0.0 -0.0229 0.0 rpy=0.0 0.0 0.0, axis 0 0 1, limit lower=0.0 upper=1.57 effort=10 velocity=1
- added joint rightPelvisIMU_Offset: type fixed, parent pelvis, child rightPelvisIMU_Frame, origin xyz=0.0515 -0.115 -0.042 rpy=-1.57 0.0 1.274, axis 0 0 1
- added joint rightPinkyPitch1: type revolute, parent rightPalm, child rightPinkyPitch1Link, origin xyz=0.0022 -0.0838 -0.041 rpy=0.1222 0.0 0.0, axis 0 0 1, limit lower=0.0 upper=1.57 effort=10 velocity=1
- added joint rightPinkyPitch2: type revolute, parent rightPinkyPitch1Link, child rightPinkyPitch2Link, origin xyz=0.0 -0.0381 0.0 rpy=0.0 0.0 0.0, axis 0 0 1, limit lower=0.0 upper=1.658 effort=10 velocity=1
- added joint rightPinkyPitch3: type revolute, parent rightPinkyPitch2Link, child rightPinkyPitch3Link, origin xyz=0.0 -0.0229 0.0 rpy=0.0 0.0 0.0, axis 0 0 1, limit lower=0.0 upper=1.92 effort=10 velocity=1
- added joint rightShoulderPitch: type revolute, parent torso, child rightShoulderPitchLink, origin xyz=-0.0316 0.0 0.2984 rpy=0.0 0.0 0.0, axis 0 1 0, limit lower=-2.85 upper=2.0 effort=190 velocity=5.89
- added joint rightShoulderRoll: type revolute, parent rightShoulderPitchLink, child rightShoulderRollLink, origin xyz=0.0 -0.2499 0.0 rpy=0.0 0.0 0.0, axis 1 0 0, limit lower=-1.266 upper=1.519 effort=190 velocity=5.89
- added joint rightShoulderYaw: type revolute, parent rightShoulderRollLink, child rightShoulderYawLink, origin xyz=0.0 0.0 0.0 rpy=0.0 0.0 0.0, axis 0 1 0, limit lower=-3.1 upper=2.18 effort=65 velocity=11.5
- added joint rightThumbPitch1: type revolute, parent rightThumbRollLink, child rightThumbPitch1Link, origin xyz=0.0 0.0 0.0229 rpy=-0.3491 0.0 0.0, axis 1 0 0, limit lower=0.0 upper=1.658 effort=10 velocity=1
- added joint rightThumbPitch2: type revolute, parent rightThumbPitch1Link, child rightThumbPitch2Link, origin xyz=0.0 -0.0066 0.0375 rpy=0.0 0.0 0.0, axis 1 0 0, limit lower=0.0 upper=1.92 effort=10 velocity=1
- added joint rightThumbPitch3: type revolute, parent rightThumbPitch2Link, child rightThumbPitch3Link, origin xyz=0.0 -0.0049 0.0275 rpy=0.0 0.0 0.0, axis 1 0 0, limit lower=0.0 upper=1.57 effort=10 velocity=1
- added joint rightThumbRoll: type revolute, parent rightPalm, child rightThumbRollLink, origin xyz=0.0049 -0.0351 0.0228 rpy=0.3491 0.0 0.0, axis 0 1 0, limit lower=0.0 upper=2.356 effort=10 velocity=1
- added joint rightTorsoIMU_Offset: type fixed, parent torso, child rightTorsoIMU_Frame, origin xyz=-0.047 -0.134 0.363 rpy=-1.57 0.0 3.14, axis 0 0 1
- added joint rightWristPitch: type revolute, parent rightWristRollLink, child rightPalm, origin xyz=0.0 0.0 0.0 rpy=0.0 0.0 0.0, axis 0 0 1, limit lower=-0.49 upper=0.36 effort=14 velocity=1
- added joint rightWristRoll: type revolute, parent rightForearmLink, child rightWristRollLink, origin xyz=0.0 -0.2871 0.0 rpy=0.0 0.0 0.0, axis 1 0 0, limit lower=-0.625 upper=0.62 effort=14 velocity=1
- added joint torsoPitch: type revolute, parent torsoYawLink, child torsoPitchLink, origin xyz=0.04191 0.0 0.0 rpy=0.0 0.0 0.0, axis 0 1 0, limit lower=-0.13 upper=0.666 effort=150 velocity=9
- added joint torsoRoll: type revolute, parent torsoPitchLink, child torso, origin xyz=0.0 0.0 0.0203 rpy=0.0 0.0 0.0, axis 1 0 0, limit lower=-0.23 upper=0.255 effort=150 velocity=9
- added joint torsoYaw: type revolute, parent pelvis, child torsoYawLink, origin xyz=0.0 0.0 0.0 rpy=0.0 0.0 0.0, axis 0 0 1, limit lower=-1.329 upper=1.181 effort=190 velocity=5.89
- added joint upperNeckPitch: type revolute, parent neckYawLink, child upperNeckPitchLink, origin xyz=-0.06 0 0.195997 rpy=0.0 0.0 0.0, axis 0 1 0, limit lower=-0.872 upper=0.0 effort=26 velocity=5
- joint multisense_head_root_joint: parent UpperNeckPitchLink -> upperNeckPitchLink
