Commit message: ROSI-258: Update model files

File: resources/models/val_description/model/robots/common/xacro/pelvis/pelvis.xacro (robot description, xacro)
@@ -18,6 +18,19 @@
         <xacro:microstrain_sensor sensorName="pelvisMiddleImu"
                                   parentLink="${Pelvis_Link_Name}"
-                                  origin_xyz="0.0 0.0 -0.108184035"
-                                  origin_rpy="3.14159 0.0 0.0" />
+                                  origin_xyz="0.012 0.0 -0.108184035"
+                                  origin_rpy="3.14159 0.0 -3.14159" />
+    </xacro:macro>
+    <xacro:macro name="v1_pelvis_sensors_usb" params="sensor_node_tag sensor_api_tag sensor_port_tag">
+        <xacro:microstrain_sensor sensorName="pelvisRearImu"
+                                  parentLink="${Pelvis_Link_Name}"
+                                  origin_xyz="-0.075844901 0.0 -0.111056426"
+                                  origin_rpy="-3.14159 0.476467 -3.14159" />
+        <xacro:usb_microstrain_sensor sensorName="pelvisMiddleImu"
+                                  parentLink="${Pelvis_Link_Name}"
+                                  origin_xyz="0.012 0.0 -0.108184035"
+                                  origin_rpy="3.14159 0.0 -3.14159"
+                                  sensor_node="${sensor_node_tag}"
+                                  sensor_api="${sensor_api_tag}"
+                                  sensor_port="${sensor_port_tag}" />
     </xacro:macro>
 </robot>

File: resources/models/val_description/urdf/valkyrie_A_hw.urdf (robot description, URDF)
Before this commit: robot valkyrie_A_hw, 67 links, 66 joints
Joints:
- joint pelvisMiddleImu_Offset: origin xyz=0.0 0.0 -0.108184035 rpy=3.14159 0.0 0.0 -> xyz=0.012 0.0 -0.108184035 rpy=3.14159 0.0 -3.14159

File: resources/models/val_description/urdf/valkyrie_A_no_hands_hw.urdf (robot description, URDF)
Before this commit: robot valkyrie_A_no_hands_hw, 35 links, 34 joints
Joints:
- joint pelvisMiddleImu_Offset: origin xyz=0.0 0.0 -0.108184035 rpy=3.14159 0.0 0.0 -> xyz=0.012 0.0 -0.108184035 rpy=3.14159 0.0 -3.14159

File: resources/models/val_description/urdf/valkyrie_B_hw.urdf (robot description, URDF)
Before this commit: robot valkyrie_B_hw, 67 links, 66 joints
Joints:
- joint pelvisMiddleImu_Offset: origin xyz=0.0 0.0 -0.108184035 rpy=3.14159 0.0 0.0 -> xyz=0.012 0.0 -0.108184035 rpy=3.14159 0.0 -3.14159

File: resources/models/val_description/urdf/valkyrie_B_no_hands_hw.urdf (robot description, URDF)
Before this commit: robot valkyrie_B_no_hands_hw, 35 links, 34 joints
Joints:
- joint pelvisMiddleImu_Offset: origin xyz=0.0 0.0 -0.108184035 rpy=3.14159 0.0 0.0 -> xyz=0.012 0.0 -0.108184035 rpy=3.14159 0.0 -3.14159

File: resources/models/val_description/urdf/valkyrie_C_hw.urdf (robot description, URDF)
Before this commit: robot valkyrie_C_hw, 67 links, 66 joints
Joints:
- joint pelvisMiddleImu_Offset: origin xyz=0.0 0.0 -0.108184035 rpy=3.14159 0.0 0.0 -> xyz=0.012 0.0 -0.108184035 rpy=3.14159 0.0 -3.14159

File: resources/models/val_description/urdf/valkyrie_C_no_hands_hw.urdf (robot description, URDF)
Before this commit: robot valkyrie_C_no_hands_hw, 35 links, 34 joints
Joints:
- joint pelvisMiddleImu_Offset: origin xyz=0.0 0.0 -0.108184035 rpy=3.14159 0.0 0.0 -> xyz=0.012 0.0 -0.108184035 rpy=3.14159 0.0 -3.14159

File: resources/models/val_description/urdf/valkyrie_sim.urdf (robot description, URDF)
Before this commit: robot valkyrie_sim, 78 links, 77 joints
Joints:
- joint pelvisMiddleImu_Offset: origin xyz=0.0 0.0 -0.108184035 rpy=3.14159 0.0 0.0 -> xyz=0.012 0.0 -0.108184035 rpy=3.14159 0.0 -3.14159
