Commit message: Added test to compare SDF to URDF.

File: valkyrie/src/main/resources/models/val_description/urdf/valkyrie_sim.urdf (robot description, URDF)
Before this commit: robot valkyrie, 78 links, 77 joints
Links:
- removed link center_bottom_led_frame
- removed link center_top_led_frame
- removed link head
- removed link head_hokuyo_frame
- removed link head_imu_link
- removed link hokuyo_link
- removed link left_camera_frame
- removed link left_camera_optical_frame
- removed link left_led_frame
- removed link right_camera_frame
- removed link right_camera_optical_frame
- removed link right_led_frame
- added link leftFootSixAxis_Frame, mass 1e-07
- added link multisense/head, mass 1e-07
- added link rightFootSixAxis_Frame, mass 1e-07
- added link zedm_mount, mass 1e-07
- link leftHipRollLink: geometry 
- link rightHipRollLink: geometry 
- link torso: mass 39.47 -> 30.87
Joints:
- removed joint center_bottom_led_frame_joint
- removed joint center_top_led_frame_joint
- removed joint head_hokuyo_joint
- removed joint head_imu_joint
- removed joint hokuyo_joint
- removed joint left_camera_frame_joint
- removed joint left_camera_optical_frame_joint
- removed joint left_led_frame_joint
- removed joint right_camera_frame_joint
- removed joint right_camera_optical_frame_joint
- removed joint right_led_frame_joint
- added joint leftFootSixAxis_Offset: type fixed, parent leftFoot, child leftFootSixAxis_Frame, origin xyz=0.0215646 0.0 -0.051054 rpy=3.14 0.0 0.0, axis 0 0 1
- added joint rightFootSixAxis_Offset: type fixed, parent rightFoot, child rightFootSixAxis_Frame, origin xyz=0.0215646 0.0 -0.051054 rpy=3.14 0.0 0.0, axis 0 0 1
- added joint zedm_head_root_joint: type fixed, parent upperNeckPitchLink, child zedm_mount, origin xyz=0.192184 0.0 -0.096498 rpy=0.0 0.1309 0.0, axis 0 0 1
- joint leftAnklePitch: limit lower=-0.8644 upper=0.875 effort=205 velocity=11 -> lower=-0.93 upper=0.65 effort=205 velocity=11
- joint leftAnkleRoll: limit lower=-0.349 upper=0.348 effort=205 velocity=11 -> lower=-0.4 upper=0.4 effort=205 velocity=11
- joint leftElbowPitch: limit lower=-2.174 upper=0.12 effort=65 velocity=3.5 -> lower=-2.13 upper=0.04 effort=65 velocity=11.5
- joint leftForearmYaw: limit lower=-2.019 upper=3.14 effort=26 velocity=0.8 -> lower=-2.019 upper=3.14 effort=26 velocity=5
- joint leftHipPitch: limit lower=-2.42 upper=1.619 effort=350 velocity=6.11 -> lower=-1.63 upper=1.549 effort=350 velocity=6.11
- joint leftHipRoll: limit lower=-0.467 upper=0.5515 effort=350 velocity=7 -> lower=-0.45 upper=0.4815 effort=350 velocity=7
- joint leftHipYaw: limit lower=-0.4141 upper=1.1 effort=190 velocity=5.89 -> lower=-0.38 upper=1.03 effort=190 velocity=5.89
- joint leftIndexFingerPitch1: origin xyz=0.0022 0.0976 0.0235 rpy=0.1745 0.0 0.0 -> xyz=0.0022 0.0976 0.017 rpy=-0.02 0.0 0.0
- joint leftIndexFingerPitch2: mimic (none) -> joint=leftIndexFingerPitch1 multiplier=0.835 offset=0
- joint leftIndexFingerPitch3: mimic (none) -> joint=leftIndexFingerPitch1 multiplier=0.668 offset=0
- joint leftKneePitch: limit lower=-0.083 upper=2.057 effort=350 velocity=6.11 -> lower=-0.055 upper=1.95 effort=350 velocity=6.11
- joint leftMiddleFingerPitch2: mimic (none) -> joint=leftMiddleFingerPitch1 multiplier=0.835 offset=0
- joint leftMiddleFingerPitch3: mimic (none) -> joint=leftMiddleFingerPitch1 multiplier=0.668 offset=0
- joint leftPinkyPitch1: origin xyz=0.0022 0.0838 -0.041 rpy=-0.1222 0.0 0.0 -> xyz=0.0022 0.0838 -0.041 rpy=-0.22 0.0 0.0
- joint leftPinkyPitch2: mimic (none) -> joint=leftPinkyPitch1 multiplier=0.835 offset=0
- joint leftPinkyPitch3: mimic (none) -> joint=leftPinkyPitch1 multiplier=0.668 offset=0
- joint leftShoulderPitch: limit lower=-2.85 upper=2.0 effort=190 velocity=3.0 -> lower=-2.78 upper=1.93 effort=190 velocity=5.89
- joint leftShoulderRoll: limit lower=-1.519 upper=1.266 effort=190 velocity=3.5 -> lower=-1.449 upper=1.196 effort=190 velocity=5.89
- joint leftShoulderYaw: limit lower=-3.1 upper=2.18 effort=65 velocity=1.5 -> lower=-3.03 upper=3.03 effort=65 velocity=11.5
- joint leftThumbPitch2: mimic (none) -> joint=leftThumbPitch1 multiplier=0.835 offset=0
- joint leftThumbPitch3: mimic (none) -> joint=leftThumbPitch1 multiplier=0.668 offset=0
- joint leftWristPitch: limit lower=-0.36 upper=0.49 effort=14 velocity=1 -> lower=-0.6 upper=0.6 effort=14 velocity=1
- joint leftWristRoll: limit lower=-0.62 upper=0.625 effort=14 velocity=1 -> lower=-0.35 upper=0.35 effort=14 velocity=1
- joint multisense_head_root_joint: child head -> multisense/head
- joint rightAnklePitch: limit lower=-0.8644 upper=0.875 effort=205 velocity=11 -> lower=-0.93 upper=0.65 effort=205 velocity=11
- joint rightAnkleRoll: limit lower=-0.349 upper=0.348 effort=205 velocity=11 -> lower=-0.4 upper=0.4 effort=205 velocity=11
- joint rightElbowPitch: limit lower=-0.12 upper=2.174 effort=65 velocity=3.5 -> lower=-0.04 upper=2.13 effort=65 velocity=11.5
- joint rightForearmYaw: limit lower=-2.019 upper=3.14 effort=26 velocity=0.8 -> lower=-2.019 upper=3.14 effort=26 velocity=5
- joint rightHipPitch: limit lower=-2.42 upper=1.619 effort=350 velocity=6.11 -> lower=-1.63 upper=1.549 effort=350 velocity=6.11
- joint rightHipRoll: limit lower=-0.5515 upper=0.467 effort=350 velocity=7 -> lower=-0.4815 upper=0.45 effort=350 velocity=7
- joint rightHipYaw: limit lower=-1.1 upper=0.4141 effort=190 velocity=5.89 -> lower=-1.03 upper=0.38 effort=190 velocity=5.89
- joint rightIndexFingerPitch1: origin xyz=0.0022 -0.0976 0.0235 rpy=-0.1745 0.0 0.0 -> xyz=0.0022 -0.0976 0.017 rpy=0.02 0.0 0.0
- joint rightIndexFingerPitch2: mimic (none) -> joint=rightIndexFingerPitch1 multiplier=0.835 offset=0
- joint rightIndexFingerPitch3: mimic (none) -> joint=rightIndexFingerPitch1 multiplier=0.668 offset=0
- joint rightKneePitch: limit lower=-0.083 upper=2.057 effort=350 velocity=6.11 -> lower=-0.055 upper=1.95 effort=350 velocity=6.11
- joint rightMiddleFingerPitch2: mimic (none) -> joint=rightMiddleFingerPitch1 multiplier=0.835 offset=0
- joint rightMiddleFingerPitch3: mimic (none) -> joint=rightMiddleFingerPitch1 multiplier=0.668 offset=0
- joint rightPinkyPitch1: origin xyz=0.0022 -0.0838 -0.041 rpy=0.1222 0.0 0.0 -> xyz=0.0022 -0.0838 -0.041 rpy=0.22 0.0 0.0
- joint rightPinkyPitch2: mimic (none) -> joint=rightPinkyPitch1 multiplier=0.835 offset=0
- joint rightPinkyPitch3: mimic (none) -> joint=rightPinkyPitch1 multiplier=0.668 offset=0
- joint rightShoulderPitch: limit lower=-2.85 upper=2.0 effort=190 velocity=3.0 -> lower=-2.78 upper=1.93 effort=190 velocity=5.89
- joint rightShoulderRoll: limit lower=-1.266 upper=1.519 effort=190 velocity=3.5 -> lower=-1.196 upper=1.449 effort=190 velocity=5.89
- joint rightShoulderYaw: limit lower=-3.1 upper=2.18 effort=65 velocity=1.5 -> lower=-3.03 upper=3.03 effort=65 velocity=11.5
- joint rightThumbPitch2: mimic (none) -> joint=rightThumbPitch1 multiplier=0.835 offset=0
- joint rightThumbPitch3: mimic (none) -> joint=rightThumbPitch1 multiplier=0.668 offset=0
- joint rightWristPitch: limit lower=-0.49 upper=0.36 effort=14 velocity=1 -> lower=-0.6 upper=0.6 effort=14 velocity=1
- joint rightWristRoll: limit lower=-0.625 upper=0.62 effort=14 velocity=1 -> lower=-0.35 upper=0.35 effort=14 velocity=1
- joint torsoYaw: limit lower=-1.329 upper=1.181 effort=190 velocity=5.89 -> lower=-1.259 upper=1.111 effort=190 velocity=5.89

Commit message: Reduced the diff between JSC URDF and IHMC SDF

File: valkyrie/src/main/resources/models/val_description/urdf/valkyrie_sim.urdf (robot description, URDF)
Before this commit: robot valkyrie, 70 links, 69 joints
Joints:
- joint leftAnklePitch: limit lower=-0.93 upper=0.65 effort=205 velocity=11 -> lower=-0.8644 upper=0.875 effort=205 velocity=11
- joint leftAnkleRoll: limit lower=-0.4 upper=0.4 effort=205 velocity=11 -> lower=-0.349 upper=0.348 effort=205 velocity=11; origin xyz=0.0 0.0 0.0 rpy=0.0 0.0 0.0 -> xyz=0.0101259 0.0 0.0 rpy=0.0 0.0 0.0
- joint leftElbowPitch: limit lower=-2.13 upper=0.04 effort=65 velocity=11.5 -> lower=-2.174 upper=0.12 effort=65 velocity=3.5
- joint leftForearmYaw: limit lower=-2.019 upper=3.14 effort=26 velocity=5 -> lower=-2.019 upper=3.14 effort=26 velocity=0.8
- joint leftHipPitch: limit lower=-1.63 upper=1.549 effort=350 velocity=6.11 -> lower=-2.42 upper=1.619 effort=350 velocity=6.11
- joint leftHipRoll: limit lower=-0.45 upper=0.4815 effort=350 velocity=7 -> lower=-0.467 upper=0.5515 effort=350 velocity=7
- joint leftHipYaw: limit lower=-0.38 upper=1.03 effort=190 velocity=5.89 -> lower=-0.4141 upper=1.10 effort=190 velocity=5.89
- joint leftKneePitch: limit lower=-0.055 upper=1.95 effort=350 velocity=6.11 -> lower=-0.083 upper=2.057 effort=350 velocity=6.11
- joint leftShoulderPitch: limit lower=-2.78 upper=1.93 effort=190 velocity=5.89 -> lower=-2.85 upper=2.00 effort=190 velocity=3
- joint leftShoulderRoll: limit lower=-1.449 upper=1.196 effort=190 velocity=5.89 -> lower=-1.519 upper=1.266 effort=350 velocity=3.5
- joint leftShoulderYaw: limit lower=-3.03 upper=3.03 effort=65 velocity=11.5 -> lower=-3.10 upper=2.18 effort=65 velocity=1.5
- joint rightAnklePitch: limit lower=-0.93 upper=0.65 effort=205 velocity=11 -> lower=-0.8644 upper=0.875 effort=205 velocity=11
- joint rightAnkleRoll: limit lower=-0.4 upper=0.4 effort=205 velocity=11 -> lower=-0.349 upper=0.348 effort=205 velocity=11; origin xyz=0.0 0.0 0.0 rpy=0.0 0.0 0.0 -> xyz=0.0101259 0.0 0.0 rpy=0.0 0.0 0.0
- joint rightElbowPitch: limit lower=-0.04 upper=2.13 effort=65 velocity=11.5 -> lower=-0.12 upper=2.174 effort=65 velocity=3.5
- joint rightForearmYaw: limit lower=-2.019 upper=3.14 effort=26 velocity=5 -> lower=-2.019 upper=3.14 effort=26 velocity=0.8
- joint rightHipPitch: limit lower=-1.63 upper=1.549 effort=350 velocity=6.11 -> lower=-2.42 upper=1.619 effort=350 velocity=6.11
- joint rightHipRoll: limit lower=-0.4815 upper=0.45 effort=350 velocity=7 -> lower=-0.5515 upper=0.467 effort=350 velocity=7
- joint rightHipYaw: limit lower=-1.03 upper=0.38 effort=190 velocity=5.89 -> lower=-1.10 upper=0.4141 effort=190 velocity=5.89
- joint rightKneePitch: limit lower=-0.055 upper=1.95 effort=350 velocity=6.11 -> lower=-0.083 upper=2.057 effort=350 velocity=6.11
- joint rightShoulderPitch: limit lower=-2.78 upper=1.93 effort=190 velocity=5.89 -> lower=-2.85 upper=2.0 effort=190 velocity=3
- joint rightShoulderRoll: limit lower=-1.196 upper=1.449 effort=190 velocity=5.89 -> lower=-1.266 upper=1.519 effort=350 velocity=3.5
- joint rightShoulderYaw: limit lower=-3.03 upper=3.03 effort=65 velocity=11.5 -> lower=-3.10 upper=2.18 effort=65 velocity=1.5
- joint torsoYaw: limit lower=-1.259 upper=1.111 effort=190 velocity=5.89 -> lower=-1.329 upper=1.181 effort=190 velocity=5.89

Commit message: Added the multisense head

File: valkyrie/src/main/resources/models/val_description/urdf/valkyrie_sim.urdf (robot description, URDF)
Before this commit: robot valkyrie, 70 links, 69 joints
Links:
- added link center_bottom_led_frame, mass 1e-5
- added link center_top_led_frame, mass 1e-5
- added link head_hokuyo_frame, mass 1e-5
- added link head_imu_link, mass 1e-5
- added link hokuyo_link, mass 0.057654; collision box size=0.08 0.06 0.04238; collision cylinder length=0.047 radius=0.024425
- added link left_camera_frame, mass 1e-5
- added link left_camera_optical_frame
- added link left_led_frame, mass 1e-5
- added link right_camera_frame, mass 1e-5
- added link right_camera_optical_frame
- added link right_led_frame, mass 1e-5
- link multisense/head: mass 1e-07 -> 1.41984; geometry collision box size=0.0468 0.12 0.1184; collision box size=0.1311 0.12 0.0591
Joints:
- added joint center_bottom_led_frame_joint: type fixed, parent multisense/head, child center_bottom_led_frame, origin xyz=0.01125 0.0 -0.0155
- added joint center_top_led_frame_joint: type fixed, parent multisense/head, child center_top_led_frame, origin xyz=0.01125 0.0 0.0105
- added joint head_hokuyo_joint: type fixed, parent hokuyo_link, child head_hokuyo_frame, origin xyz=0.03 0 0.015 rpy=0 0 0, axis 0 1 0
- added joint head_imu_joint: type fixed, parent multisense/head, child head_imu_link, origin xyz=-0.0475 0.035 0.0 rpy=0 0 0
- added joint hokuyo_joint: type revolute, parent multisense/head, child hokuyo_link, origin xyz=-0.0446 0 0.0880 rpy=0 0 0, axis 1 0 0, limit lower=-1e+16 upper=1e+16
- added joint left_camera_frame_joint: type fixed, parent multisense/head, child left_camera_frame, origin xyz=0.0 0.035 -0.002
- added joint left_camera_optical_frame_joint: type fixed, parent left_camera_frame, child left_camera_optical_frame, origin xyz=0 0 0 rpy=-1.5708 0.0 -1.5708
- added joint left_led_frame_joint: type fixed, parent multisense/head, child left_led_frame, origin xyz=-0.01443 0.07452 0.050346 rpy=0 -0.15 0.53
- added joint right_camera_frame_joint: type fixed, parent multisense/head, child right_camera_frame, origin xyz=0.0 -0.035 -0.002
- added joint right_camera_optical_frame_joint: type fixed, parent right_camera_frame, child right_camera_optical_frame, origin xyz=0 0 0 rpy=-1.5708 0.0 -1.5708
- added joint right_led_frame_joint: type fixed, parent multisense/head, child right_led_frame, origin xyz=-0.01443 -0.07452 0.050346 rpy=0 -0.15 -0.53

File: valkyrie/src/main/resources/models/val_description/urdf/valkyrie_sim_arm_mass_sim.urdf (robot description, URDF)
Before this commit: robot valkyrie, 38 links, 37 joints
Links:
- added link center_bottom_led_frame, mass 1e-5
- added link center_top_led_frame, mass 1e-5
- added link head_hokuyo_frame, mass 1e-5
- added link head_imu_link, mass 1e-5
- added link hokuyo_link, mass 0.057654; collision box size=0.08 0.06 0.04238; collision cylinder length=0.047 radius=0.024425
- added link left_camera_frame, mass 1e-5
- added link left_camera_optical_frame
- added link left_led_frame, mass 1e-5
- added link right_camera_frame, mass 1e-5
- added link right_camera_optical_frame
- added link right_led_frame, mass 1e-5
- link multisense/head: mass 1e-07 -> 1.41984; geometry collision box size=0.0468 0.12 0.1184; collision box size=0.1311 0.12 0.0591
Joints:
- added joint center_bottom_led_frame_joint: type fixed, parent multisense/head, child center_bottom_led_frame, origin xyz=0.01125 0.0 -0.0155
- added joint center_top_led_frame_joint: type fixed, parent multisense/head, child center_top_led_frame, origin xyz=0.01125 0.0 0.0105
- added joint head_hokuyo_joint: type fixed, parent hokuyo_link, child head_hokuyo_frame, origin xyz=0.03 0 0.015 rpy=0 0 0, axis 0 1 0
- added joint head_imu_joint: type fixed, parent multisense/head, child head_imu_link, origin xyz=-0.0475 0.035 0.0 rpy=0 0 0
- added joint hokuyo_joint: type revolute, parent multisense/head, child hokuyo_link, origin xyz=-0.0446 0 0.0880 rpy=0 0 0, axis 1 0 0, limit lower=-1e+16 upper=1e+16
- added joint left_camera_frame_joint: type fixed, parent multisense/head, child left_camera_frame, origin xyz=0.0 0.035 -0.002
- added joint left_camera_optical_frame_joint: type fixed, parent left_camera_frame, child left_camera_optical_frame, origin xyz=0 0 0 rpy=-1.5708 0.0 -1.5708
- added joint left_led_frame_joint: type fixed, parent multisense/head, child left_led_frame, origin xyz=-0.01443 0.07452 0.050346 rpy=0 -0.15 0.53
- added joint right_camera_frame_joint: type fixed, parent multisense/head, child right_camera_frame, origin xyz=0.0 -0.035 -0.002
- added joint right_camera_optical_frame_joint: type fixed, parent right_camera_frame, child right_camera_optical_frame, origin xyz=0 0 0 rpy=-1.5708 0.0 -1.5708
- added joint right_led_frame_joint: type fixed, parent multisense/head, child right_led_frame, origin xyz=-0.01443 -0.07452 0.050346 rpy=0 -0.15 -0.53

File: valkyrie/src/main/resources/models/val_description/urdf/valkyrie_sim_no_arms.urdf (robot description, URDF)
Before this commit: robot valkyrie, 30 links, 29 joints
Links:
- added link center_bottom_led_frame, mass 1e-5
- added link center_top_led_frame, mass 1e-5
- added link head_hokuyo_frame, mass 1e-5
- added link head_imu_link, mass 1e-5
- added link hokuyo_link, mass 0.057654; collision box size=0.08 0.06 0.04238; collision cylinder length=0.047 radius=0.024425
- added link left_camera_frame, mass 1e-5
- added link left_camera_optical_frame
- added link left_led_frame, mass 1e-5
- added link right_camera_frame, mass 1e-5
- added link right_camera_optical_frame
- added link right_led_frame, mass 1e-5
- link multisense/head: mass 1e-07 -> 1.41984; geometry collision box size=0.0468 0.12 0.1184; collision box size=0.1311 0.12 0.0591
Joints:
- added joint center_bottom_led_frame_joint: type fixed, parent multisense/head, child center_bottom_led_frame, origin xyz=0.01125 0.0 -0.0155
- added joint center_top_led_frame_joint: type fixed, parent multisense/head, child center_top_led_frame, origin xyz=0.01125 0.0 0.0105
- added joint head_hokuyo_joint: type fixed, parent hokuyo_link, child head_hokuyo_frame, origin xyz=0.03 0 0.015 rpy=0 0 0, axis 0 1 0
- added joint head_imu_joint: type fixed, parent multisense/head, child head_imu_link, origin xyz=-0.0475 0.035 0.0 rpy=0 0 0
- added joint hokuyo_joint: type revolute, parent multisense/head, child hokuyo_link, origin xyz=-0.0446 0 0.0880 rpy=0 0 0, axis 1 0 0, limit lower=-1e+16 upper=1e+16
- added joint left_camera_frame_joint: type fixed, parent multisense/head, child left_camera_frame, origin xyz=0.0 0.035 -0.002
- added joint left_camera_optical_frame_joint: type fixed, parent left_camera_frame, child left_camera_optical_frame, origin xyz=0 0 0 rpy=-1.5708 0.0 -1.5708
- added joint left_led_frame_joint: type fixed, parent multisense/head, child left_led_frame, origin xyz=-0.01443 0.07452 0.050346 rpy=0 -0.15 0.53
- added joint right_camera_frame_joint: type fixed, parent multisense/head, child right_camera_frame, origin xyz=0.0 -0.035 -0.002
- added joint right_camera_optical_frame_joint: type fixed, parent right_camera_frame, child right_camera_optical_frame, origin xyz=0 0 0 rpy=-1.5708 0.0 -1.5708
- added joint right_led_frame_joint: type fixed, parent multisense/head, child right_led_frame, origin xyz=-0.01443 -0.07452 0.050346 rpy=0 -0.15 -0.53

File: valkyrie/src/main/resources/models/val_description/urdf/valkyrie_sim_no_fingers.urdf (robot description, URDF)
Before this commit: robot valkyrie, 44 links, 43 joints
Links:
- added link center_bottom_led_frame, mass 1e-5
- added link center_top_led_frame, mass 1e-5
- added link head_hokuyo_frame, mass 1e-5
- added link head_imu_link, mass 1e-5
- added link hokuyo_link, mass 0.057654; collision box size=0.08 0.06 0.04238; collision cylinder length=0.047 radius=0.024425
- added link left_camera_frame, mass 1e-5
- added link left_camera_optical_frame
- added link left_led_frame, mass 1e-5
- added link right_camera_frame, mass 1e-5
- added link right_camera_optical_frame
- added link right_led_frame, mass 1e-5
- link multisense/head: mass 1e-07 -> 1.41984; geometry collision box size=0.0468 0.12 0.1184; collision box size=0.1311 0.12 0.0591
Joints:
- added joint center_bottom_led_frame_joint: type fixed, parent multisense/head, child center_bottom_led_frame, origin xyz=0.01125 0.0 -0.0155
- added joint center_top_led_frame_joint: type fixed, parent multisense/head, child center_top_led_frame, origin xyz=0.01125 0.0 0.0105
- added joint head_hokuyo_joint: type fixed, parent hokuyo_link, child head_hokuyo_frame, origin xyz=0.03 0 0.015 rpy=0 0 0, axis 0 1 0
- added joint head_imu_joint: type fixed, parent multisense/head, child head_imu_link, origin xyz=-0.0475 0.035 0.0 rpy=0 0 0
- added joint hokuyo_joint: type revolute, parent multisense/head, child hokuyo_link, origin xyz=-0.0446 0 0.0880 rpy=0 0 0, axis 1 0 0, limit lower=-1e+16 upper=1e+16
- added joint left_camera_frame_joint: type fixed, parent multisense/head, child left_camera_frame, origin xyz=0.0 0.035 -0.002
- added joint left_camera_optical_frame_joint: type fixed, parent left_camera_frame, child left_camera_optical_frame, origin xyz=0 0 0 rpy=-1.5708 0.0 -1.5708
- added joint left_led_frame_joint: type fixed, parent multisense/head, child left_led_frame, origin xyz=-0.01443 0.07452 0.050346 rpy=0 -0.15 0.53
- added joint right_camera_frame_joint: type fixed, parent multisense/head, child right_camera_frame, origin xyz=0.0 -0.035 -0.002
- added joint right_camera_optical_frame_joint: type fixed, parent right_camera_frame, child right_camera_optical_frame, origin xyz=0 0 0 rpy=-1.5708 0.0 -1.5708
- added joint right_led_frame_joint: type fixed, parent multisense/head, child right_led_frame, origin xyz=-0.01443 -0.07452 0.050346 rpy=0 -0.15 -0.53
