Commit message: moved most of the atlas end to end controller api tests, swapping for alexander

File: open-alexander/src/main/resources/models/alexander_v0/urdf/alexander_v0.lowerBody.urdf (robot description, URDF)
Before this commit: robot alexander, 18 links, 17 joints
Joints:
- joint NECK_Y: type fixed -> revolute
- joint NECK_Z: type fixed -> revolute

Commit message: Alexander lowerbody urdf is replaced with new one. each meshes files are updated.

File: open-alexander/src/main/resources/models/alexander_v0/urdf/alexander_v0.lowerBody.urdf (robot description, URDF)
Before this commit: robot alexander, 18 links, 17 joints
Links:
- added link LEFT_FOOT_IMU_LINK, mass 0
- added link LEFT_HIP_X_IMU_LINK, mass 0
- added link LEFT_SHIN_IMU_LINK, mass 0
- added link LEFT_THIGH_IMU_LINK, mass 0
- added link RIGHT_FOOT_IMU_LINK, mass 0
- added link RIGHT_HIP_X_IMU_LINK, mass 0
- added link RIGHT_SHIN_IMU_LINK, mass 0
- added link RIGHT_THIGH_IMU_LINK, mass 0
- link LEFT_ANKLE_Y_LINK: mass 0.19 -> 0.05045632; geometry visual mesh filename=package://alexander_v0/meshes/legs//AnklePitchLink.obj
- link LEFT_FOOT: mass 1.01 -> 1.28288609; geometry visual mesh filename=package://alexander_v0/meshes/legs//Foot.obj
- link LEFT_HIP_X_LINK: mass 2.48 -> 2.32977961; geometry visual mesh filename=package://alexander_v0/meshes/legs//LeftHipRollLink.obj
- link LEFT_HIP_Z_LINK: mass 0.70 -> 0.77281362; geometry visual mesh filename=package://alexander_v0/meshes/legs//LeftHipYawLink.obj
- link LEFT_SHIN: mass 7.68 -> 5.5; geometry visual mesh filename=package://alexander_v0/meshes/legs//LeftShin.obj
- link LEFT_THIGH: mass 7.57 -> 7.75; geometry visual mesh filename=package://alexander_v0/meshes/legs//LeftThigh.obj
- link PELVIS_LINK: mass 9.55 -> 9.50083635; geometry visual mesh filename=package://alexander_v0/meshes/legs//Pelvis.obj
- link RIGHT_ANKLE_Y_LINK: mass 0.19 -> 0.05045632; geometry visual mesh filename=package://alexander_v0/meshes/legs//AnklePitchLink.obj
- link RIGHT_FOOT: mass 1.01 -> 1.28288609; geometry visual mesh filename=package://alexander_v0/meshes/legs//Foot.obj
- link RIGHT_HIP_X_LINK: mass 2.48 -> 2.32977248; geometry visual mesh filename=package://alexander_v0/meshes/legs//RightHipRollLink.obj
- link RIGHT_HIP_Z_LINK: mass 0.70 -> 0.77281055; geometry visual mesh filename=package://alexander_v0/meshes/legs//RightHipYawLink.obj
- link RIGHT_SHIN: mass 7.68 -> 5.5; geometry visual mesh filename=package://alexander_v0/meshes/legs//RightShin.obj
- link RIGHT_THIGH: mass 7.57 -> 7.75; geometry visual mesh filename=package://alexander_v0/meshes/legs//RightThigh.obj
- link TORSO_LINK: mass 13.5 -> 4.208
Joints:
- added joint LEFT_FOOT_IMU_JOINT: type fixed, parent LEFT_FOOT, child LEFT_FOOT_IMU_LINK, origin xyz=-0.03575526 0.01180178 -0.04979705 rpy=0 0 1.570796, axis 0 0 1
- added joint LEFT_HIP_X_IMU_JOINT: type fixed, parent LEFT_HIP_X_LINK, child LEFT_HIP_X_IMU_LINK, origin xyz=-0.01922309 0.10145013 -0.01488788 rpy=-1.570796 0 1.570796, axis 0 0 1
- added joint LEFT_SHIN_IMU_JOINT: type fixed, parent LEFT_SHIN, child LEFT_SHIN_IMU_LINK, origin xyz=0.05655120 0.00084826 -0.15664831 rpy=1.403695170631842 0 -1.570796, axis 0 0 1
- added joint LEFT_THIGH_IMU_JOINT: type fixed, parent LEFT_THIGH, child LEFT_THIGH_IMU_LINK, origin xyz=0.10004 0.03746 -0.21194 rpy=1.6947717585 0 1.570796, axis 0 0 1
- added joint RIGHT_FOOT_IMU_JOINT: type fixed, parent RIGHT_FOOT, child RIGHT_FOOT_IMU_LINK, origin xyz=-0.03575526 0.01180178 -0.04979705 rpy=0 0 1.570796, axis 0 0 1
- added joint RIGHT_HIP_ROLL_IMU_JOINT: type fixed, parent RIGHT_HIP_X_LINK, child RIGHT_HIP_X_IMU_LINK, origin xyz=-0.01922309 -0.07694987 -0.01488788 rpy=-1.570796 0 1.570796, axis 0 0 1
- added joint RIGHT_SHIN_IMU_JOINT: type fixed, parent RIGHT_SHIN, child RIGHT_SHIN_IMU_LINK, origin xyz=0.05673025 -0.00875818 -0.15674961 rpy=1.403695170631842 0 -1.570796, axis 0 0 1
- added joint RIGHT_THIGH_IMU_JOINT: type fixed, parent RIGHT_THIGH, child RIGHT_THIGH_IMU_LINK, origin xyz=0.10003618 -0.033541826 -0.21194191 rpy=1.6947717585 0 1.570796, axis 0 0 1
- joint LEFT_ANKLE_X: origin xyz=0 0 -0.01 rpy=0 0 0 -> xyz=0 0 -0.012 rpy=0 0 0
- joint LEFT_HIP_X: limit lower=-1.0472 upper=0.436332 effort=150 velocity=9 -> lower=-0.3490658504  upper=0.872664626 effort=150 velocity=9; origin xyz=-0.16935 0.056 -0.01485 rpy=0 0 0 -> xyz=-0.162 0.0595 -0.015 rpy=0 0 0
- joint LEFT_HIP_Y: origin xyz=0.098 -0.046 -0.045 rpy=0 0 0 -> xyz=0.1045 -0.0573 -0.0525 rpy=0 0 0
- joint LEFT_HIP_Z: origin xyz=0.05 0.0965 -0.072 rpy=0 0 0 -> xyz=0.06 0.1 -0.08 rpy=0 0 0
- joint LEFT_KNEE_Y: limit lower=0 upper=2.61799 effort=200 velocity=8 -> lower=0 upper=2.445206282 effort=200 velocity=8; origin xyz=0 0.015 -0.32 rpy=0 0 0 -> xyz=0 0.018 -0.32 rpy=0 0 0
- joint PELVIS_STIM_IMU_JOINT: origin xyz=-0.03133646 0.02237500 -0.07000000 rpy=0.0 3.141592 0.0 -> xyz=-0.08687724 0.01225028 -0.08051472 rpy=0.0 0.0 1.570796
- joint RIGHT_ANKLE_X: origin xyz=0 0 -0.01 rpy=0 0 0 -> xyz=0 0 -0.012 rpy=0 0 0
- joint RIGHT_HIP_X: limit lower=-0.436332 upper=1.0472 effort=150 velocity=9 -> lower=-0.872664626 upper=0.3490658504 effort=150 velocity=9; origin xyz=-0.16935 -0.056 -0.01485 rpy=0 0 0 -> xyz=-0.162 -0.0595 -0.015 rpy=0 0 0
- joint RIGHT_HIP_Y: origin xyz=0.098 0.046 -0.045 rpy=0 0 0 -> xyz=0.1045 0.0573 -0.0525 rpy=0 0 0
- joint RIGHT_HIP_Z: origin xyz=0.05 -0.0965 -0.072 rpy=0 0 0 -> xyz=0.06 -0.1 -0.08 rpy=0 0 0
- joint RIGHT_KNEE_Y: limit lower=0 upper=2.61799 effort=200 velocity=8 -> lower=0 upper=2.445206282 effort=200 velocity=8; origin xyz=0 -0.015 -0.32 rpy=0 0 0 -> xyz=0 -0.018 -0.32 rpy=0 0 0
- joint SPINE_Z: limit lower=-1.570796327 upper=1.570796327 effort=150 velocity=9.0 -> lower=-0.5235987756 upper=0.5235987756 effort=150 velocity=9.0; origin xyz=0.005 0 0.0785 rpy=0 0 0 -> xyz=0.0 0 0.018 rpy=0 0 0
