Commit message: Cleaned up the resources paths to be shorter and easier, made sure the robot model gets logged properly

File: zulu/src/main/resources/zulu/urdf/zulu-full-body.urdf (robot description, URDF)
Before this commit: robot Zulu, 51 links, 50 joints
Links:
- link HEAD_LINK: geometry collision sphere radius=0.13; visual mesh filename=package://zulu/meshes/ALX02_01_A02_HeadLink.obj
- link LEFT_ANKLE_Y_LINK: geometry visual mesh filename=package://zulu/meshes/legs/AnklePitchLink.obj
- link LEFT_ELBOW_Y_LINK: geometry visual mesh filename=package://zulu/meshes/cycloidal_arm/LeftElbowPitchLink.obj
- link LEFT_FOOT: geometry collision box size=0.22 0.1 0.02; visual mesh filename=package://zulu/meshes/legs/Foot.obj
- link LEFT_GRIPPER_ATTACHMENT_FIXED_LINK: geometry visual mesh filename=package://zulu/meshes/wristmesh.obj
- link LEFT_GRIPPER_Z_LINK: geometry collision sphere radius=0.05; visual mesh filename=package://zulu/meshes/cycloidal_arm/nub.obj
- link LEFT_HIP_X_LINK: geometry collision box size=0.02 0.12 0.10; visual mesh filename=package://zulu/meshes/legs/LeftHipRollLink.obj
- link LEFT_HIP_Z_LINK: geometry visual mesh filename=package://zulu/meshes/legs/LeftHipYawLink.obj
- link LEFT_SHIN: geometry collision cylinder length=0.3 radius=0.08; visual mesh filename=package://zulu/meshes/legs/LeftShin.obj
- link LEFT_SHOULDER_X_LINK: geometry visual mesh filename=package://zulu/meshes/cycloidal_arm/LeftShoulderRollLink_sh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
- link LEFT_SHOULDER_Y_LINK: geometry visual mesh filename=package://zulu/meshes/cycloidal_arm/LeftShoulderPitchLink.o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
- link LEFT_SHOULDER_Z_LINK: geometry collision cylinder length=0.15 radius=0.05; visual mesh filename=package://zulu/meshes/cycloidal_arm/LeftShoulderYawLink.obj
- link LEFT_THIGH: geometry collision box size=0.16 0.13 0.29; visual mesh filename=package://zulu/meshes/legs/LeftThigh.obj
- link LEFT_WRIST_X_LINK: geometry visual mesh filename=package://zulu/meshes/cycloidal_arm/LeftWristRollLink.obj
- link LEFT_WRIST_Z_LINK: geometry collision box size=0.01 0.06 0.1; collision cylinder length=0.12 radius=0.044
- link PELVIS_LINK: geometry collision box size=0.15 0.10 0.12; visual mesh filename=package://zulu/meshes/legs/Pelvis.obj
- link RIGHT_ANKLE_Y_LINK: geometry visual mesh filename=package://zulu/meshes/legs/AnklePitchLink.obj
- link RIGHT_ELBOW_Y_LINK: geometry visual mesh filename=package://zulu/meshes/cycloidal_arm/RightElbowPitchLink.obj
- link RIGHT_FOOT: geometry collision box size=0.22 0.1 0.02; visual mesh filename=package://zulu/meshes/legs/Foot.obj
- link RIGHT_GRIPPER_ATTACHMENT_FIXED_LINK: geometry visual mesh filename=package://zulu/meshes/wristmesh.obj
- link RIGHT_GRIPPER_Z_LINK: geometry collision sphere radius=0.05; visual mesh filename=package://zulu/meshes/cycloidal_arm/nub.obj
- link RIGHT_HIP_X_LINK: geometry collision box size=0.02 0.12 0.10; visual mesh filename=package://zulu/meshes/legs/RightHipRollLink.obj
- link RIGHT_HIP_Z_LINK: geometry visual mesh filename=package://zulu/meshes/legs/RightHipYawLink.obj
- link RIGHT_SHIN: geometry collision cylinder length=0.3 radius=0.08; visual mesh filename=package://zulu/meshes/legs/RightShin.obj
- link RIGHT_SHOULDER_X_LINK: geometry visual mesh filename=package://zulu/meshes/cycloidal_arm/RightShoulderRollLink_s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
- link RIGHT_SHOULDER_Y_LINK: geometry visual mesh filename=package://zulu/meshes/cycloidal_arm/RightShoulderPitchLink.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
- link RIGHT_SHOULDER_Z_LINK: geometry collision cylinder length=0.15 radius=0.05; visual mesh filename=package://zulu/meshes/cycloidal_arm/RightShoulderYawLink.obj
- link RIGHT_THIGH: geometry collision box size=0.16 0.13 0.29; visual mesh filename=package://zulu/meshes/legs/RightThigh.obj
- link RIGHT_WRIST_X_LINK: geometry visual mesh filename=package://zulu/meshes/cycloidal_arm/RightWristRollLink.obj
- link RIGHT_WRIST_Z_LINK: geometry collision box size=0.01 0.06 0.1; collision cylinder length=0.12 radius=0.044
- link TORSO_LINK: geometry collision box size=0.275 0.33 0.43; visual mesh filename=package://zulu/meshes/torso.obj

Commit message: Shorted file path name for mesh's

File: zulu/src/main/resources/zulu/urdf/zulu-full-body.urdf (robot description, URDF)
Before this commit: robot Zulu, 51 links, 50 joints
Links:
- link HEAD_LINK: geometry collision sphere radius=0.13; visual mesh filename=zulu/meshes/ALX02_01_A02_HeadLink.obj
- link LEFT_ANKLE_Y_LINK: geometry visual mesh filename=zulu/meshes/legs/AnklePitchLink.obj
- link LEFT_ELBOW_Y_LINK: geometry visual mesh filename=zulu/meshes/cycloidal_arm/LeftElbowPitchLink.obj
- link LEFT_FOOT: geometry collision box size=0.22 0.1 0.02; visual mesh filename=zulu/meshes/legs/Foot.obj
- link LEFT_GRIPPER_ATTACHMENT_FIXED_LINK: geometry visual mesh filename=zulu/meshes/wristmesh.obj
- link LEFT_GRIPPER_Z_LINK: geometry collision sphere radius=0.05; visual mesh filename=zulu/meshes/cycloidal_arm/nub.obj
- link LEFT_HIP_X_LINK: geometry collision box size=0.02 0.12 0.10; visual mesh filename=zulu/meshes/legs/LeftHipRollLink.obj
- link LEFT_HIP_Z_LINK: geometry visual mesh filename=zulu/meshes/legs/LeftHipYawLink.obj
- link LEFT_SHIN: geometry collision cylinder length=0.3 radius=0.08; visual mesh filename=zulu/meshes/legs/LeftShin.obj
- link LEFT_SHOULDER_X_LINK: geometry visual mesh filename=zulu/meshes/cycloidal_arm/LeftShoulderRollLink_shortBicep.o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
- link LEFT_SHOULDER_Y_LINK: geometry visual mesh filename=zulu/meshes/cycloidal_arm/LeftShoulderPitchLink.obj
- link LEFT_SHOULDER_Z_LINK: geometry collision cylinder length=0.15 radius=0.05; visual mesh filename=zulu/meshes/cycloidal_arm/LeftShoulderYawLink.obj
- link LEFT_THIGH: geometry collision box size=0.16 0.13 0.29; visual mesh filename=zulu/meshes/legs/LeftThigh.obj
- link LEFT_WRIST_X_LINK: geometry visual mesh filename=zulu/meshes/cycloidal_arm/LeftWristRollLink.obj
- link LEFT_WRIST_Z_LINK: geometry collision box size=0.01 0.06 0.1; collision cylinder length=0.12 radius=0.044
- link PELVIS_LINK: geometry collision box size=0.15 0.10 0.12; visual mesh filename=zulu/meshes/legs/Pelvis.obj
- link RIGHT_ANKLE_Y_LINK: geometry visual mesh filename=zulu/meshes/legs/AnklePitchLink.obj
- link RIGHT_ELBOW_Y_LINK: geometry visual mesh filename=zulu/meshes/cycloidal_arm/RightElbowPitchLink.obj
- link RIGHT_FOOT: geometry collision box size=0.22 0.1 0.02; visual mesh filename=zulu/meshes/legs/Foot.obj
- link RIGHT_GRIPPER_ATTACHMENT_FIXED_LINK: geometry visual mesh filename=zulu/meshes/wristmesh.obj
- link RIGHT_GRIPPER_Z_LINK: geometry collision sphere radius=0.05; visual mesh filename=zulu/meshes/cycloidal_arm/nub.obj
- link RIGHT_HIP_X_LINK: geometry collision box size=0.02 0.12 0.10; visual mesh filename=zulu/meshes/legs/RightHipRollLink.obj
- link RIGHT_HIP_Z_LINK: geometry visual mesh filename=zulu/meshes/legs/RightHipYawLink.obj
- link RIGHT_SHIN: geometry collision cylinder length=0.3 radius=0.08; visual mesh filename=zulu/meshes/legs/RightShin.obj
- link RIGHT_SHOULDER_X_LINK: geometry visual mesh filename=zulu/meshes/cycloidal_arm/RightShoulderRollLink_shortBicep.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
- link RIGHT_SHOULDER_Y_LINK: geometry visual mesh filename=zulu/meshes/cycloidal_arm/RightShoulderPitchLink.obj
- link RIGHT_SHOULDER_Z_LINK: geometry collision cylinder length=0.15 radius=0.05; visual mesh filename=zulu/meshes/cycloidal_arm/RightShoulderYawLink.obj
- link RIGHT_THIGH: geometry collision box size=0.16 0.13 0.29; visual mesh filename=zulu/meshes/legs/RightThigh.obj
- link RIGHT_WRIST_X_LINK: geometry visual mesh filename=zulu/meshes/cycloidal_arm/RightWristRollLink.obj
- link RIGHT_WRIST_Z_LINK: geometry collision box size=0.01 0.06 0.1; collision cylinder length=0.12 radius=0.044
- link TORSO_LINK: geometry collision box size=0.275 0.33 0.43; visual mesh filename=zulu/meshes/torso.obj

Commit message: Do xyz first, then rpy, match convention for loading URDF

File: zulu/src/main/resources/zulu/urdf/zulu-full-body.urdf (robot description, URDF)
Before this commit: robot Zulu, 51 links, 50 joints
Joints:
- joint LEFT_ANKLE_X: origin xyz=0 0 -0.012 rpy=0 0 0 -> xyz=0 0 0 rpy=0 0 -0.012
- joint LEFT_ANKLE_Y: origin xyz=0 0 -0.41 rpy=0 0 0 -> xyz=0 0 0 rpy=0 0 -0.41
- joint LEFT_HIP_X: origin xyz=-0.162 0.0595 -0.015 rpy=0 0 0 -> xyz=0 0 0 rpy=-0.162 0.0595 -0.015
- joint LEFT_HIP_Y: origin xyz=0.1045 -0.0573 -0.0525 rpy=0 0 0 -> xyz=0 0 0 rpy=0.1045 -0.0573 -0.0525
- joint LEFT_HIP_Z: origin xyz=0.06 0.1 -0.08 rpy=0 0 0 -> xyz=0 0 0 rpy=0.06 0.1 -0.08
- joint LEFT_KNEE_Y: origin xyz=0 0.018 -0.32 rpy=0 0 0 -> xyz=0 0 0 rpy=0 0.018 -0.32
- joint NECK_Y: origin xyz=0.025 0.01 0.189597 rpy=0 0 0 -> xyz=0 0 0 rpy=0.025 0.01 0.189597
- joint NECK_Z: origin xyz=-0.015 0 0.450403 rpy=0 0 0 -> xyz=0 0 0 rpy=-0.015 0 0.450403
- joint RIGHT_ANKLE_X: origin xyz=0 0 -0.012 rpy=0 0 0 -> xyz=0 0 0 rpy=0 0 -0.012
- joint RIGHT_ANKLE_Y: origin xyz=0 0 -0.41 rpy=0 0 0 -> xyz=0 0 0 rpy=0 0 -0.41
- joint RIGHT_HIP_X: origin xyz=-0.162 -0.0595 -0.015 rpy=0 0 0 -> xyz=0 0 0 rpy=-0.162 -0.0595 -0.015
- joint RIGHT_HIP_Y: origin xyz=0.1045 0.0573 -0.0525 rpy=0 0 0 -> xyz=0 0 0 rpy=0.1045 0.0573 -0.0525
- joint RIGHT_HIP_Z: origin xyz=0.06 -0.1 -0.08 rpy=0 0 0 -> xyz=0 0 0 rpy=0.06 -0.1 -0.08
- joint RIGHT_KNEE_Y: origin xyz=0 -0.018 -0.32 rpy=0 0 0 -> xyz=0 0 0 rpy=0 -0.018 -0.32
- joint SPINE_Z: origin xyz=0.0 0 0.018 rpy=0 0 0 -> xyz=0 0 0 rpy=0.0 0 0.018

Commit message: Cleanup URDF

File: zulu/src/main/resources/zulu/urdf/zulu-full-body.urdf (robot description, URDF)
Before this commit: robot Zulu, 51 links, 50 joints
Joints:
- joint HEAD_IMU_JOINT: origin xyz=0.040556 -0.014155 0.057016 rpy=0.56723 0.0 1.5708  -> xyz=0.040556 -0.014155 0.057016 rpy=0.56723 0.0 1.5708
