Commit message: Update the ZuluPhysicalProperties

File: zulu/src/main/resources/us/ihmc/zulu/urdf/zulu-full-body.urdf (robot description, URDF)
Before this commit: robot Zulu, 51 links, 50 joints
Joints:
- joint LEFT_ANKLE_X: limit lower=-0.436332 upper=0.436332 effort=180 velocity=8 -> lower=-0.436332 upper=0.436332 effort=145.2 velocity=9.72
- joint LEFT_ANKLE_Y: limit lower=-1.0472 upper=0.523599 effort=360 velocity=8 -> lower=-1.0472 upper=0.523599 effort=193.6 velocity=9.72
- joint LEFT_HIP_X: limit lower=-0.3490658504 upper=0.872664626 effort=300 velocity=9 -> lower=-0.3490658504 upper=0.872664626 effort=160.7 velocity=10.38
- joint LEFT_HIP_Y: limit lower=-2.61799 upper=0.785398 effort=400 velocity=8 -> lower=-2.61799 upper=0.785398 effort=217.2 velocity=9.3
- joint LEFT_HIP_Z: limit lower=-0.3490658504 upper=1.0472 effort=120 velocity=11 -> lower=-0.3490658504 upper=1.0472 effort=70.5 velocity=10.59
- joint LEFT_KNEE_Y: limit lower=0 upper=2.445206282 effort=400 velocity=8 -> lower=0 upper=2.445206282 effort=217.2 velocity=9.3
- joint RIGHT_ANKLE_X: limit lower=-0.436332 upper=0.436332 effort=180 velocity=8 -> lower=-0.436332 upper=0.436332 effort=145.2 velocity=9.72
- joint RIGHT_ANKLE_Y: limit lower=-1.0472 upper=0.523599 effort=360 velocity=8 -> lower=-1.0472 upper=0.523599 effort=193.6 velocity=9.72
- joint RIGHT_HIP_X: limit lower=-0.872664626 upper=0.3490658504 effort=300 velocity=9 -> lower=-0.872664626 upper=0.3490658504 effort=160.7 velocity=10.38
- joint RIGHT_HIP_Y: limit lower=-2.61799 upper=0.785398 effort=400 velocity=8 -> lower=-2.61799 upper=0.785398 effort=217.2 velocity=9.3
- joint RIGHT_HIP_Z: limit lower=-1.0472 upper=0.3490658504 effort=120 velocity=11 -> lower=-1.0472 upper=0.3490658504 effort=70.5 velocity=10.59
- joint RIGHT_KNEE_Y: limit lower=0 upper=2.445206282 effort=400 velocity=8 -> lower=0 upper=2.445206282 effort=217.2 velocity=9.3

Commit message: More changes to match the real robot

File: zulu/src/main/resources/us/ihmc/zulu/urdf/zulu-full-body.urdf (robot description, URDF)
Before this commit: robot Zulu, 51 links, 50 joints
Links:
- link LEFT_FOOT: mass 1.28288609 -> 0.810
- link LEFT_HIP_X_LINK: mass 2.32977961 -> 2.33165613
- link LEFT_HIP_Z_LINK: mass 0.77281362 -> 0.761264535
- link LEFT_SHIN: mass 6.31087157 -> 6.33845554
- link LEFT_THIGH: mass 7.75 -> 8.281087115
- link PELVIS_LINK: mass 9.50083635 -> 7.161
- link RIGHT_FOOT: mass 1.28288609 -> 0.810
- link RIGHT_HIP_X_LINK: mass 2.32977248 -> 2.33165613
- link RIGHT_HIP_Z_LINK: mass 0.77281055 -> 0.761264535
- link RIGHT_SHIN: mass 6.31087157 -> 6.33845554
- link RIGHT_THIGH: mass 7.75 -> 8.281087115

Commit message: More changes to match the real robot

File: zulu/src/main/resources/us/ihmc/zulu/urdf/zulu-full-body.urdf (robot description, URDF)
Before this commit: robot Zulu, 51 links, 50 joints
Links:
- link LEFT_SHOULDER_X_LINK: mass 0.972 -> 1.16159753
- link LEFT_SHOULDER_Y_LINK: mass 2.99 -> 3.02036119
- link LEFT_SHOULDER_Z_LINK: mass 2.91 -> 3.117556435
- link RIGHT_SHOULDER_X_LINK: mass 0.972 -> 1.16159753
- link RIGHT_SHOULDER_Y_LINK: mass 2.99 -> 3.02036119
- link RIGHT_SHOULDER_Z_LINK: mass 2.91 -> 3.117556435

Commit message: More changes to match the real robot

File: zulu/src/main/resources/us/ihmc/zulu/urdf/zulu-full-body.urdf (robot description, URDF)
Before this commit: robot Zulu, 51 links, 50 joints
Links:
- link TORSO_LINK: mass 7.0081 -> 22.210
